File: Bipolar_transistor_tester_1.0/Bipolar_transistor_tester_1.0.kicad_pcb (KiCad board)
At the start: 2 copper layers, 203 parts, among them IC1 OPA454, IC2 OPA454, IC3 OPA454, IC4 OPA454, IC5 OPA454, J1 KF2510_7pin, J10 DJ621-6.3, J11 DJ621-6.3, J12 DJ621-6.3, J13 DJ621-6.3, J14 DJ621-6.3, J15 DJ621-6.3, J16 DJ621-6.3, J2 KF2510_6pin, J3 DJ621-6.3, J4 DJ621-6.3, J5 DJ621-6.3, J6 DJ621-6.3, J7 DJ621-6.3, J8 DJ621-6.3, J9 DJ621-6.3, Q1 AO3400A, Q2 AO3401A, Q3 IRFR9024 [DPAK], Q4 IRF640 [DPAK], Q5 AO3400A, Q6 AO3401A, Q7 IRFR9024 [DPAK], Q8 IRF640 [DPAK], U1 CPC1977, U10 PVN012, U11 CPC1977, U12 CPC1977, U13 PVN012, U14 PVN012, U15 PVN012, U16 PVN012, U17 INA118, U18 ISO124P, U19 PVN012, U2 PVN012, U20 PVN012, U21 AD549, U22 CPC1977, U23 PVG612, U24 PVN012, U25 OP07, U26 PVN012, U27 PVN012, U28 PVN012, U29 PVN012, U3 AD822, U30 PVN012, U31 CPC1977, U32 PVG612, U33 CPC1977, U34 CPC1977, U35 AD822, U36 PVN012, U37 PVN012, U38 PVN012, U39 PVN012, U4 PVN012, U40 PVN012, U41 PVN012, U42 PVN012, U43 PVG612, U44 PVG612, U45 PVG612, U46 PVG612, U47 PVG612, U48 INA118, U5 PVN012, U6 PVN012, U7 PVN012, U8 PVN012, U9 PVN012

Commit message: tester up
Parts:
- added H1: MountingHole, MountingHole:MountingHole_3.2mm_M3, F.Cu at (34.0, 18.0)
- added H2: MountingHole, MountingHole:MountingHole_3.2mm_M3, F.Cu at (34.0, 68.0)
- added H3: MountingHole, MountingHole:MountingHole_3.2mm_M3, F.Cu at (196.0, 18.0)
- added H4: MountingHole, MountingHole:MountingHole_3.2mm_M3, F.Cu at (196.0, 68.0)
- added H5: MountingHole, MountingHole:MountingHole_3.2mm_M3, F.Cu at (34.0, 150.0)
- added H6: MountingHole, MountingHole:MountingHole_3.2mm_M3, F.Cu at (196.0, 150.0)
- added J17: KF2510_2pin, Connector_KF2510:KF2510_2pin, F.Cu at (187.4, 148.8)
- added J18: KF2510_2pin, Connector_KF2510:KF2510_2pin, F.Cu at (152.1, 63.7)
- added J19: KF2510_5pin, Connector_KF2510:KF2510_5pin, F.Cu at (139.8, 120.1)
- added J20: KF2510_5pin, Connector_KF2510:KF2510_5pin, F.Cu at (111.0, 24.4)
- added J21: KF2510_6pin, Connector_KF2510:KF2510_6pin, F.Cu at (55.3, 147.3)
- added J22: KF2510_4pin, Connector_KF2510:KF2510_4pin, F.Cu at (187.2, 77.4)
- added J23: KF2510_2pin, Connector_KF2510:KF2510_2pin, F.Cu at (179.1, 92.0)
- added J24: KF2510_2pin, Connector_KF2510:KF2510_2pin, F.Cu at (149.7, 147.0)
- added J25: DJ621-6.3, Connector:Knife_Terminal_6.3mm_P5.00mm_Vertical, F.Cu at (155.5, 24.1)
- added J26: DJ621-6.3, Connector:Knife_Terminal_6.3mm_P5.00mm_Vertical, F.Cu at (185.0, 24.1)
- added J27: DJ621-6.3, Connector:Knife_Terminal_6.3mm_P5.00mm_Vertical, F.Cu at (155.8, 37.3)
- added J28: DJ621-6.3, Connector:Knife_Terminal_6.3mm_P5.00mm_Vertical, F.Cu at (185.5, 37.2)
- added J29: DJ621-6.3, Connector:Knife_Terminal_6.3mm_P5.00mm_Vertical, F.Cu at (156.0, 50.9)
- added R100: 1k 1%, Resistor_SMD:R_0805_2012Metric, B.Cu at (127.3, 139.8)
- added R101: 51k 1%, Resistor_SMD:R_0805_2012Metric, B.Cu at (138.5, 139.5)
- added R102: 100, Resistor_SMD:R_0805_2012Metric, B.Cu at (146.0, 144.2)
- added R79: 10 1% 0.5W, Resistor_THT:R_Axial_DIN0309_L9.0mm_D3.2mm_P12.70mm_Horizontal, F.Cu at (91.4, 132.8)
- added R80: 1k 1%, Resistor_SMD:R_0805_2012Metric, B.Cu at (82.1, 114.5)
- added R81: 1k 1%, Resistor_SMD:R_0805_2012Metric, B.Cu at (81.7, 123.9)
- added R82: 2.2k, Resistor_SMD:R_0805_2012Metric, B.Cu at (57.8, 114.4)
- added R83: 2.2k, Resistor_SMD:R_0805_2012Metric, B.Cu at (74.3, 129.1)
- added R84: 20k 1%, Resistor_SMD:R_0805_2012Metric, B.Cu at (98.1, 110.4)
- added R85: 20k 1%, Resistor_SMD:R_0805_2012Metric, B.Cu at (95.6, 129.4)
- added R86: 1k 1%, Resistor_SMD:R_0805_2012Metric, B.Cu at (92.9, 114.6)
- added R87: 1k 1%, Resistor_SMD:R_0805_2012Metric, B.Cu at (92.9, 124.0)
- added R88: 20M 1%, Resistor_SMD:R_0805_2012Metric, B.Cu at (108.8, 110.4)
- added R89: 20M 1%, Resistor_SMD:R_0805_2012Metric, B.Cu at (106.4, 128.9)
- added R90: 1k 1%, Resistor_SMD:R_0805_2012Metric, B.Cu at (103.6, 114.7)
- added R91: 1k 1%, Resistor_SMD:R_0805_2012Metric, B.Cu at (103.4, 124.0)
- added R92: 1k 1%, Resistor_SMD:R_0805_2012Metric, B.Cu at (113.3, 106.6)
- added R93: 10M 1%, Resistor_SMD:R_0805_2012Metric, B.Cu at (123.1, 103.8)
- added R94: 1k 1%, Resistor_SMD:R_0805_2012Metric, B.Cu at (127.2, 108.8)
- added R95: 100k 1%, Resistor_SMD:R_0805_2012Metric, B.Cu at (123.2, 114.0)
- added R96: 1k 1%, Resistor_SMD:R_0805_2012Metric, B.Cu at (127.4, 119.2)
- added R97: 1k 1%, Resistor_SMD:R_0805_2012Metric, B.Cu at (123.2, 124.2)
- added R98: 1k 1%, Resistor_SMD:R_0805_2012Metric, B.Cu at (127.4, 129.4)
- added R99: 5 1% 0.5W, Resistor_THT:R_Axial_DIN0309_L9.0mm_D3.2mm_P12.70mm_Horizontal, F.Cu at (122.3, 134.4)
- C1, C17, C18, C19, C2, C20, C21, C22, C23, C24, C25, C26, C27, C28, C29, C3, C30, C31, C32, C4, C5, C6, C7, C8, C9, IC1, IC2, IC3, IC4, IC5, Q1, Q2, Q5, Q6, R2, R25, R26, R33, R38, R46, R48, R52, R54, R61, R66, R67, R7, R72, R75, R8: moved to B.Cu
- J10, J11, J3, J4, J5, J6, J7, J8, J9: footprint Connector:CONN_63824-1 -> Connector:Knife_Terminal_6.3mm_P5.00mm_Vertical
- J12: value DJ621-6.3 -> KF2510_3pin; footprint Connector:CONN_63824-1 -> Connector_KF2510:KF2510_3pin
- J13, J14: value DJ621-6.3 -> KF2510_6pin; footprint Connector:CONN_63824-1 -> Connector_KF2510:KF2510_6pin
- J15, J16: value DJ621-6.3 -> KF2510_5pin; footprint Connector:CONN_63824-1 -> Connector_KF2510:KF2510_5pin
- Q3, Q7: value IRFR9024 [DPAK] -> IRFR9024; moved to B.Cu
- Q4, Q8: value IRF640 [DPAK] -> IRF640; moved to B.Cu
- R1: value 100k -> 1k 1%; moved to B.Cu
- R10, R56, R57, R9: value 51k -> 1k 1%; moved to B.Cu
- R11, R12: value 2 1% -> 51k; moved to B.Cu
- R13, R14: value 1k 1% -> 2 1% 0.5W; footprint Resistor_SMD:R_0805_2012Metric -> Resistor_THT:R_Axial_DIN0309_L9.0mm_D3.2mm_P12.70mm_Horizontal
- R15, R16: value 2.2k -> 1k 1%; moved to B.Cu
- R17, R18: value 200 1% -> 2.2k; moved to B.Cu
- R19, R20: value 1k 1% -> 200 1%; moved to B.Cu
- R21, R22: value 10k 1% -> 1k 1%; moved to B.Cu
- R23, R24: value 1k 1% -> 10k 1%; moved to B.Cu
- R27: value 0,1 1% -> 1k 1%; moved to B.Cu
- R28, R58: value 10 1% -> 1k 1%; moved to B.Cu
- R29: value 1k 1% -> 0,1 1% 0.5W; footprint Resistor_SMD:R_0805_2012Metric -> Resistor_THT:R_Axial_DIN0309_L9.0mm_D3.2mm_P12.70mm_Horizontal
- R3: value 270 -> 100k; moved to B.Cu
- R30, R74: value 100k 1% -> 1k 1%; moved to B.Cu
- R31: value 2k 1% -> 10 1% 0.5W; footprint Resistor_SMD:R_0805_2012Metric -> Resistor_THT:R_Axial_DIN0309_L9.0mm_D3.2mm_P12.70mm_Horizontal
- R32, R41: value 100 -> 1k 1%; moved to B.Cu
- R34: value 100M 1% -> 1k 1%; moved to B.Cu
- R35: value 100 -> 100k 1%; moved to B.Cu
- R36, R45: value 1M 1% -> 1k 1%; moved to B.Cu
- R37: value 200k 1% -> 2k 1%; moved to B.Cu
- R39: value 1 -> 1k 1%; moved to B.Cu
- R4, R50: value 270 -> 1k 1%; moved to B.Cu
- R40: value 10 -> 1k 1%; moved to B.Cu
- R42: value 1k -> 100M 1%; moved to B.Cu
- R43: value 200k -> 100; moved to B.Cu
- R44: value 200k -> 1k 1%; moved to B.Cu
- R47: value 100k -> 200k 1%; moved to B.Cu
- R49: value 100k -> 100; moved to B.Cu
- R5, R6, R70, R71: value 1k 1% -> 270; moved to B.Cu
- R51: value 270 -> 1 1%; moved to B.Cu
- R53: value 1k 1% -> 10 1%; moved to B.Cu
- R55: value 1k 1% -> 100 1%; moved to B.Cu
- R59: value 10 1% -> 200k; moved to B.Cu
- R60: value 1k 1% -> 200k; moved to B.Cu
- R62, R63: value 2.2k -> 1M 1%; moved to B.Cu
- R64: value 200k 1% -> 100k; moved to B.Cu
- R65: value 200k 1% -> 1k 1%; moved to B.Cu
- R68: value 20M 1% -> 1k 1%; moved to B.Cu
- R69: value 20M 1% -> 100k; moved to B.Cu
- R73: value 10M 1% -> 1k 1%; moved to B.Cu
- R76: value 5 1% -> 51k; moved to B.Cu
- R77: value 51k 1% -> 51k; moved to B.Cu
- R78: value 100 -> 10 1% 0.5W; footprint Resistor_SMD:R_0805_2012Metric -> Resistor_THT:R_Axial_DIN0309_L9.0mm_D3.2mm_P12.70mm_Horizontal
- U33: value CPC1977 -> PVG612; footprint OptoDevice:i4-PAC -> Package_DIP:DIP-6_W7.62mm
- moved R73 222.0 mm to (43.5, 127.9), turned to 180 degrees
- moved R74 206.2 mm to (57.5, 133.6)
- moved R75 197.1 mm to (61.7, 126.6)
- moved R76 196.5 mm to (57.9, 117.4), turned to 270 degrees
- moved R77 191.9 mm to (74.3, 132.6), turned to 270 degrees
- moved J7 183.6 mm to (49.2, 21.6)
- moved J5 181.2 mm to (49.2, 35.2)
- moved C24 171.9 mm to (112.2, 48.1), turned to 180 degrees
- moved C10 170.6 mm to (45.5, 47.6)
- moved R78 168.4 mm to (90.7, 107.0), turned to 180 degrees
- moved J6 167.2 mm to (49.2, 28.4)
- moved IC3 158.0 mm to (117.8, 45.1)
- moved C14 157.5 mm to (56.5, 47.6)
- moved C25 156.9 mm to (125.1, 47.1), turned to 270 degrees
- moved J11 153.1 mm to (78.2, 26.6)
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Connections:
- J12 pad 1: /measured transistor/coll_supp -> GND
- J12 pad 2: (no net) -> dac0
- J13 pad 1: /collector_base_voltage_meter/coll_in -> 1_com_an
- J13 pad 2: (no net) -> 1_ccs1
- J14 pad 1: /measured transistor/base_supp -> 2_com_an
- J14 pad 2: (no net) -> 2_bcs1
- J15 pad 1: /collector_base_voltage_meter/base_in -> 3_com_an
- J15 pad 2: (no net) -> 3_ccm1
- J16 pad 1: /measured transistor/emitter -> 4_com_an
- J16 pad 2: (no net) -> 4_ecm1
- J8 pad 1: (no net) -> +12V
- R1 pad 1: Net-(R1-Pad1) -> 4_com_an
- R1 pad 2: GND -> Net-(R1-Pad2)
- R10 pad 1: +24V -> Net-(IC2-Pad3)
- R10 pad 2: Net-(D4-Pad1) -> -24V
- R11 pad 1: Net-(R11-Pad1) -> +24V
- R11 pad 2: Net-(D5-Pad1) -> Net-(D3-Pad1)
- R12 pad 1: Net-(R12-Pad1) -> +24V
- R12 pad 2: Net-(D6-Pad2) -> Net-(D4-Pad1)
- R13 pad 1: 1_com_an -> Net-(R13-Pad1)
- R13 pad 2: Net-(R13-Pad2) -> Net-(D5-Pad1)
- R14 pad 1: 1_com_an -> Net-(D6-Pad2)
- R15 pad 1: Net-(D5-Pad2) -> 1_com_an
- R15 pad 2: Net-(IC1-Pad6) -> Net-(R15-Pad2)
- R16 pad 1: Net-(D6-Pad1) -> 1_com_an
- R16 pad 2: Net-(IC2-Pad6) -> Net-(R16-Pad2)
- R17 pad 1: Net-(R17-Pad1) -> Net-(D5-Pad2)
- R17 pad 2: Net-(D5-Pad1) -> Net-(IC1-Pad6)
- R18 pad 1: Net-(R18-Pad1) -> Net-(D6-Pad1)
- R18 pad 2: Net-(D6-Pad2) -> Net-(IC2-Pad6)
- R19 pad 1: 1_com_an -> Net-(R19-Pad1)
- R19 pad 2: Net-(R19-Pad2) -> Net-(D5-Pad1)
- R2 pad 1: 1_com_an -> 4_com_an
- R20 pad 1: 1_com_an -> Net-(R20-Pad1)
- R20 pad 2: (no net) -> Net-(D6-Pad2)
- R21 pad 1: Net-(R21-Pad1) -> 1_com_an
- R21 pad 2: Net-(D5-Pad1) -> Net-(R21-Pad2)
- R22 pad 1: Net-(R22-Pad1) -> 1_com_an
- R22 pad 2: Net-(D6-Pad2) -> Net-(R22-Pad2)
- R23 pad 1: 1_com_an -> Net-(R23-Pad1)
- R23 pad 2: Net-(R23-Pad2) -> Net-(D5-Pad1)
- R24 pad 1: 1_com_an -> Net-(R24-Pad1)
- R24 pad 2: Net-(R24-Pad2) -> Net-(D6-Pad2)
- R27 pad 1: /connectors/40v-500v -> 1_com_an
- R28 pad 1: /connectors/40v-500v -> 1_com_an
- R3 pad 1: Net-(D1-Pad1) -> Net-(R3-Pad1)
- R3 pad 2: Net-(R3-Pad2) -> GND
- R30 pad 1: /connectors/40v-500v -> Net-(R30-Pad1)
- R30 pad 2: Net-(R30-Pad2) -> 3_com_an
- R31 pad 1: Net-(R31-Pad1) -> /connectors/40v-500v
- R32 pad 1: adc0 -> Net-(R32-Pad1)
- R32 pad 2: Net-(R32-Pad2) -> 3_com_an
- R33 pad 1: Net-(C19-Pad2) -> /connectors/40v-500v
- R34 pad 1: Net-(C19-Pad2) -> Net-(R34-Pad1)
- R34 pad 2: Net-(R34-Pad2) -> 3_com_an
- R35 pad 1: adc1 -> /connectors/40v-500v
- R35 pad 2: Net-(C19-Pad2) -> Net-(R35-Pad2)
- R36 pad 2: Net-(R36-Pad2) -> 3_com_an
- R37 pad 1: Net-(R36-Pad1) -> Net-(R37-Pad1)
- R37 pad 2: GND -> Net-(R37-Pad2)
- R38 pad 1: Net-(R38-Pad1) -> adc0
- R38 pad 2: adc2 -> Net-(R38-Pad2)
- R39 pad 1: /base_resistors/in -> Net-(R39-Pad1)
- R39 pad 2: Net-(R39-Pad2) -> 4_com_an
- R4 pad 1: Net-(D2-Pad2) -> 1_com_an
- R40 pad 1: /base_resistors/in -> Net-(R40-Pad1)
- R40 pad 2: Net-(R40-Pad2) -> 4_com_an
- R41 pad 1: /base_resistors/in -> Net-(C19-Pad2)
- R42 pad 1: /base_resistors/in -> Net-(C19-Pad2)
- R43 pad 1: Net-(IC3-Pad2) -> adc1
- R43 pad 2: GND -> Net-(C19-Pad2)
- R44 pad 1: Net-(IC3-Pad3) -> 8_com_an
- R44 pad 2: dac1 -> Net-(R44-Pad2)
- R45 pad 1: Net-(IC3-Pad3) -> 8_com_an
- R45 pad 2: GND -> Net-(R45-Pad2)
- R46 pad 2: Net-(IC3-Pad2) -> Net-(R46-Pad2)
- R47 pad 1: +45V -> Net-(R46-Pad1)
- R47 pad 2: Net-(D7-Pad1) -> GND
- R48 pad 1: 2_com_an -> 8_com_an
- R49 pad 2: GND -> adc2
- R5 pad 1: +15V -> Net-(D1-Pad1)
- R5 pad 2: Net-(IC1-Pad3) -> Net-(R5-Pad2)
- R50 pad 1: Net-(D8-Pad1) -> Net-(R50-Pad1)
- R50 pad 2: Net-(R50-Pad2) -> 7_com_an
- R51 pad 1: Net-(D9-Pad2) -> /base_resistors/in
- R52 pad 1: +15V -> Net-(R52-Pad1)
- R52 pad 2: Net-(IC4-Pad3) -> 7_com_an
- R53 pad 1: Net-(D8-Pad2) -> /base_resistors/in
- R53 pad 2: GND -> Net-(R53-Pad2)
- R54 pad 1: GND -> Net-(R54-Pad1)
- R54 pad 2: Net-(D9-Pad1) -> 7_com_an
- R55 pad 1: Net-(IC5-Pad3) -> /base_resistors/in
- R55 pad 2: -15V -> Net-(R55-Pad2)
- R56 pad 1: +24V -> Net-(R56-Pad1)
- R56 pad 2: Net-(D10-Pad1) -> 7_com_an
- R57 pad 1: +24V -> /base_resistors/in
- R57 pad 2: Net-(D11-Pad1) -> Net-(R57-Pad2)
- R58 pad 2: Net-(D12-Pad1) -> 7_com_an
- R59 pad 1: Net-(R59-Pad1) -> Net-(IC3-Pad2)
- R59 pad 2: Net-(D13-Pad2) -> GND
- R6 pad 1: Net-(D1-Pad2) -> Net-(D2-Pad2)
- R6 pad 2: GND -> Net-(R6-Pad2)
- R60 pad 1: 2_com_an -> Net-(IC3-Pad3)
- R60 pad 2: Net-(R60-Pad2) -> dac1
- R61 pad 1: 2_com_an -> Net-(R61-Pad1)
- R61 pad 2: Net-(R61-Pad2) -> 6_com_an
- R62 pad 1: Net-(D12-Pad2) -> Net-(IC3-Pad3)
- R62 pad 2: Net-(IC4-Pad6) -> GND
- R63 pad 1: Net-(D13-Pad1) -> Net-(R63-Pad1)
- R63 pad 2: Net-(IC5-Pad6) -> Net-(IC3-Pad2)
- R64 pad 1: Net-(R64-Pad1) -> +45V
- R64 pad 2: Net-(D12-Pad1) -> Net-(D7-Pad1)
- R65 pad 2: Net-(D13-Pad2) -> 6_com_an
- R66 pad 1: 2_com_an -> Net-(R66-Pad1)
- R66 pad 2: Net-(R66-Pad2) -> 6_com_an
- R67 pad 1: 2_com_an -> Net-(R67-Pad1)
- R67 pad 2: Net-(R67-Pad2) -> 6_com_an
- R68 pad 1: Net-(R68-Pad1) -> 2_com_an
- R68 pad 2: Net-(D12-Pad1) -> Net-(R68-Pad2)
- R69 pad 2: Net-(D13-Pad2) -> GND
- R7 pad 1: GND -> +24V
- R7 pad 2: Net-(D2-Pad1) -> Net-(IC1-Pad3)
- R70 pad 1: 2_com_an -> Net-(D8-Pad1)
- R71 pad 1: 2_com_an -> Net-(D9-Pad2)
- R72 pad 1: 2_com_an -> +24V
- R72 pad 2: Net-(R72-Pad2) -> Net-(IC4-Pad3)
- R73 pad 1: Net-(R73-Pad1) -> Net-(D8-Pad2)
- R73 pad 2: /base_current_meter/in+ -> GND
- R74 pad 1: Net-(R74-Pad1) -> GND
- R74 pad 2: /base_current_meter/in+ -> Net-(D9-Pad1)
- R75 pad 1: Net-(R75-Pad1) -> Net-(IC5-Pad3)
- R75 pad 2: /base_current_meter/in+ -> -24V
- R76 pad 1: Net-(R76-Pad1) -> +24V
- R76 pad 2: /base_current_meter/in+ -> Net-(D10-Pad1)
- R77 pad 1: Net-(R77-Pad1) -> +24V
- R77 pad 2: Net-(R77-Pad2) -> Net-(D11-Pad1)
- R78 pad 2: adc3 -> Net-(D12-Pad1)
- R8 pad 1: Net-(IC2-Pad3) -> Net-(D1-Pad2)
- R8 pad 2: -15V -> GND
- R9 pad 1: +24V -> GND
- R9 pad 2: Net-(D3-Pad1) -> Net-(D2-Pad1)
- U1 pad 3: (no net) -> 4_rp1
- U1 pad 4: (no net) -> Net-(R1-Pad2)
- U10 pad 1: Net-(R24-Pad2) -> Net-(R26-Pad2)
- U10 pad 6: Net-(R22-Pad1) -> Net-(R24-Pad1)
- U11 pad 4: Net-(R25-Pad2) -> Net-(R27-Pad2)
- U12 pad 4: Net-(R26-Pad2) -> Net-(R28-Pad2)
- U13 pad 1: (no net) -> Net-(R30-Pad1)
- U13 pad 2: (no net) -> 3_ccm1
- U13 pad 6: Net-(R27-Pad2) -> Net-(R29-Pad2)
- U14 pad 1: (no net) -> Net-(R32-Pad1)
- U14 pad 2: (no net) -> 3_ccm2
- U14 pad 6: Net-(R28-Pad2) -> Net-(R31-Pad2)
- U15 pad 1: (no net) -> Net-(R34-Pad1)
- U15 pad 2: (no net) -> 3_ccm3
- U15 pad 6: Net-(R29-Pad2) -> Net-(R33-Pad2)
- U16 pad 1: (no net) -> Net-(R36-Pad1)
- U16 pad 2: (no net) -> 3_ccm4
- U16 pad 6: Net-(R30-Pad2) -> Net-(R35-Pad2)
- U17 pad 1: Net-(R31-Pad1) -> Net-(R37-Pad1)
- U17 pad 8: Net-(R31-Pad2) -> Net-(R37-Pad2)
- U18 pad 3: Net-(R32-Pad2) -> Net-(R38-Pad2)
- U19 pad 1: (no net) -> Net-(R39-Pad1)
- U19 pad 2: (no net) -> 4_ecm1
- U19 pad 4: Net-(R33-Pad2) -> Net-(R41-Pad2)
- U2 pad 1: (no net) -> Net-(R2-Pad2)
- U2 pad 2: (no net) -> 4_rp2
- U20 pad 1: (no net) -> Net-(R40-Pad1)
- U20 pad 2: (no net) -> 4_ecm2
- U20 pad 4: Net-(R34-Pad2) -> Net-(R42-Pad2)
- U22 pad 1: Net-(R36-Pad2) -> /collector_base_voltage_meter/coll_in
- U22 pad 2: /collector_base_voltage_meter/coll_in -> Net-(R46-Pad2)
- U22 pad 3: (no net) -> 8_cbvm1
- U22 pad 4: (no net) -> Net-(R44-Pad2)
- U23 pad 1: (no net) -> Net-(R45-Pad2)
- U23 pad 2: (no net) -> 8_cbvm3
- U23 pad 4: Net-(R36-Pad1) -> Net-(R46-Pad1)
- U24 pad 1: (no net) -> Net-(R48-Pad2)
- U24 pad 2: (no net) -> 8_cbvm2
- U24 pad 4: Net-(R36-Pad2) -> Net-(R46-Pad2)
- U24 pad 6: Net-(R36-Pad1) -> Net-(R46-Pad1)
- U25 pad 2: Net-(R38-Pad1) -> Net-(R49-Pad1)
- U25 pad 3: Net-(R36-Pad1) -> Net-(R46-Pad1)
- U25 pad 6: Net-(R38-Pad1) -> Net-(R49-Pad1)
- U26 pad 1: (no net) -> Net-(R50-Pad1)
- U26 pad 2: (no net) -> 7_br1
- U27 pad 1: (no net) -> Net-(R52-Pad1)
- U27 pad 2: (no net) -> 7_br2
- U27 pad 6: Net-(R39-Pad2) -> Net-(R51-Pad2)
- U28 pad 1: (no net) -> Net-(R54-Pad1)
- U28 pad 2: (no net) -> 7_br3
- U28 pad 6: Net-(R40-Pad2) -> Net-(R53-Pad2)
- U29 pad 1: (no net) -> Net-(R56-Pad1)
- U29 pad 2: (no net) -> 7_br4
- U29 pad 6: Net-(R41-Pad2) -> Net-(R55-Pad2)
- U3 pad 1: Net-(R3-Pad2) -> Net-(R5-Pad2)
- U3 pad 3: Net-(R1-Pad1) -> Net-(R3-Pad1)
- U3 pad 5: Net-(R1-Pad1) -> Net-(R3-Pad1)
- U3 pad 7: Net-(R4-Pad2) -> Net-(R6-Pad2)
- U30 pad 1: (no net) -> Net-(R58-Pad1)
- U30 pad 2: (no net) -> 7_br5
- U30 pad 6: Net-(R42-Pad2) -> Net-(R57-Pad2)
- U31 pad 1: Net-(R46-Pad1) -> Net-(R63-Pad1)
- U31 pad 3: (no net) -> 6_bvs1
- U31 pad 4: (no net) -> Net-(R61-Pad1)
- U32 pad 1: (no net) -> Net-(R65-Pad1)
- U32 pad 2: (no net) -> 6_bvs2
- U32 pad 4: Net-(R46-Pad1) -> Net-(R63-Pad1)
- U33 pad 1: (no net) -> Net-(R66-Pad1)
- U33 pad 2: (no net) -> 6_bvs4
- U33 pad 3: /base_current_meter/in+ -> (no net)
- U34 pad 1: (no net) -> /connectors/40v-500v
- U34 pad 2: (no net) -> Net-(IC3-Pad6)
- U34 pad 3: /connectors/40v-500v -> 6_bvs3
- U34 pad 4: Net-(IC3-Pad6) -> Net-(R67-Pad1)
- U35 pad 1: Net-(R50-Pad2) -> Net-(R70-Pad2)
- U35 pad 3: Net-(R49-Pad1) -> Net-(R69-Pad1)
- U35 pad 5: Net-(R49-Pad1) -> Net-(R69-Pad1)
- U35 pad 7: Net-(R51-Pad2) -> Net-(R71-Pad2)
- U36 pad 1: Net-(R48-Pad2) -> Net-(R68-Pad2)
- U36 pad 2: (no net) -> 2_bcs1
- U36 pad 6: Net-(R49-Pad1) -> Net-(R69-Pad1)
- U37 pad 1: Net-(R60-Pad2) -> Net-(R80-Pad2)
- U37 pad 6: Net-(R58-Pad1) -> Net-(R78-Pad1)
- U38 pad 1: Net-(R61-Pad2) -> Net-(R81-Pad2)
- U38 pad 6: Net-(R59-Pad1) -> Net-(R79-Pad1)
- U39 pad 1: Net-(R66-Pad2) -> Net-(R86-Pad2)
- U39 pad 6: Net-(R64-Pad1) -> Net-(R84-Pad1)
- U4 pad 1: Net-(R2-Pad2) -> Net-(R4-Pad2)
- U4 pad 2: (no net) -> 1_ccs1
- U4 pad 4: (no net) -> dac0
- U4 pad 6: Net-(R1-Pad1) -> Net-(R3-Pad1)
- U40 pad 1: Net-(R67-Pad2) -> Net-(R87-Pad2)
- U40 pad 6: Net-(R65-Pad1) -> Net-(R85-Pad1)
- U41 pad 1: Net-(R70-Pad2) -> Net-(R90-Pad2)
- U41 pad 6: Net-(R68-Pad1) -> Net-(R88-Pad1)
- U42 pad 1: Net-(R71-Pad2) -> Net-(R91-Pad2)
- U42 pad 6: Net-(R69-Pad1) -> Net-(R89-Pad1)
- U43 pad 1: Net-(R72-Pad2) -> Net-(R92-Pad2)
- U43 pad 2: (no net) -> 2_bcs5
- U44 pad 1: (no net) -> Net-(R94-Pad2)
- U44 pad 2: (no net) -> 5_bcm1
- U44 pad 6: Net-(R73-Pad1) -> Net-(R93-Pad1)
- U45 pad 1: (no net) -> Net-(R96-Pad2)
- U45 pad 2: (no net) -> 5_bcm2
- U45 pad 6: Net-(R74-Pad1) -> Net-(R95-Pad1)
- U46 pad 1: (no net) -> Net-(R98-Pad2)
- U46 pad 2: (no net) -> 5_bcm3
- U46 pad 6: Net-(R75-Pad1) -> Net-(R97-Pad1)
- U47 pad 1: (no net) -> Net-(R100-Pad2)
- U47 pad 2: (no net) -> 5_bcm4
- U47 pad 6: Net-(R76-Pad1) -> Net-(R99-Pad1)
- U48 pad 1: Net-(R77-Pad2) -> Net-(R101-Pad2)
- U48 pad 6: Net-(R78-Pad1) -> Net-(R102-Pad1)
- U48 pad 8: Net-(R77-Pad1) -> Net-(R101-Pad1)
- U5 pad 1: Net-(R13-Pad2) -> Net-(R15-Pad2)
- U5 pad 6: Net-(R11-Pad1) -> Net-(R13-Pad1)
- U6 pad 1: Net-(R14-Pad2) -> Net-(R16-Pad2)
- U6 pad 6: Net-(R12-Pad1) -> Net-(R14-Pad2)
- U7 pad 1: Net-(R19-Pad2) -> Net-(R21-Pad2)
- U7 pad 6: Net-(R17-Pad1) -> Net-(R19-Pad1)
- U8 pad 1: (no net) -> Net-(R22-Pad2)
- U8 pad 6: Net-(R18-Pad1) -> Net-(R20-Pad1)
- U9 pad 1: Net-(R23-Pad2) -> Net-(R25-Pad2)
- U9 pad 6: Net-(R21-Pad1) -> Net-(R23-Pad1)
Routing:
- net 2_com_an: track 0.00 -> 147.9 mm
- net 1_com_an: track 0.00 -> 145.0 mm
- net 4_com_an: track 0.00 -> 100.2 mm
- net Net-(D12-Pad1): track 0.00 -> 85.1 mm, vias 0 -> 3
- net /base_resistors/in: track 0.00 -> 84.7 mm
- net Net-(D5-Pad1): track 0.00 -> 84.0 mm, vias 0 -> 3
- net /connectors/40v-500v: track 0.00 -> 71.6 mm, vias 0 -> 1
- net Net-(Q3-Pad2): track 0.00 -> 67.7 mm
- net Net-(D6-Pad2): track 0.00 -> 66.1 mm, vias 0 -> 3
- net Net-(D13-Pad2): track 0.00 -> 65.6 mm, vias 0 -> 3
- net 1_ccs1: track 0.00 -> 65.0 mm
- net 2_bcs1: track 0.00 -> 64.9 mm
- net /measured transistor/emitter: track 0.00 -> 63.7 mm
- net 7_br5: track 0.00 -> 62.5 mm
- net /base_current_meter/in+: track 0.00 -> 60.8 mm
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- added copper zone on In2.Cu, net GND
Other:
- board outline added: 170 x 140 mm
- copper layers 2 -> 4
- net class Default: via_dia 0.8 -> 0.6
- net class HV added: clearance 1.2, trace_width 0.25, via_dia 0.6, via_drill 0.4

Commit message: tester up
Parts:
- added C33: 100n, Capacitor_SMD:C_0805_2012Metric, B.Cu at (202.5, 151.9)
- added C34: 1u, Capacitor_SMD:C_0805_2012Metric, B.Cu at (208.3, 151.9)
- added C35: 100n, Capacitor_SMD:C_0805_2012Metric, B.Cu at (211.0, 142.7)
- added C36: 100n, Capacitor_SMD:C_0805_2012Metric, B.Cu at (211.0, 139.0)
- moved J8 43.1 mm to (127.6, 51.2)
- moved J10 43.0 mm to (117.9, 36.6), turned to 90 degrees
- moved J9 41.8 mm to (127.5, 36.6)
- moved R33 34.8 mm to (199.8, 138.1), turned to 180 degrees
- moved C26 34.5 mm to (78.9, 149.3), turned to 0 degrees
- moved R92 34.1 mm to (144.7, 119.9)
- moved R10 34.0 mm to (92.1, 101.6), turned to 180 degrees
- moved C9 33.8 mm to (212.3, 157.5)
- moved J24 33.8 mm to (180.8, 160.3)
- moved R1 33.8 mm to (174.3, 95.9)
- moved R101 33.8 mm to (169.6, 152.8)
- moved C17 33.8 mm to (192.8, 87.7)
- moved C21 33.8 mm to (202.8, 90.0)
- moved C23 33.8 mm to (210.8, 100.6)
- moved C8 33.8 mm to (208.3, 139.0)
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Routing:
- net +15V: track 29.6 -> 412.4 mm, vias 0 -> 3
- net -15V: track 22.9 -> 370.1 mm
- net -24V: track 31.3 -> 330.4 mm, vias 0 -> 7
- net +24V: track 30.6 -> 302.9 mm, vias 0 -> 5
- net +12V: track 23.9 -> 191.6 mm
- net dac1: track 0.00 -> 165.1 mm, vias 0 -> 3
- net /connectors/40v-500v: track 71.6 -> 210.5 mm
- net /measured transistor/coll_supp: track 53.6 -> 161.9 mm
- net /collector_base_voltage_meter/coll_in: track 0.00 -> 97.1 mm
- net /base_current_meter/in+: track 60.8 -> 140.5 mm
- net +45V: track 18.2 -> 94.1 mm, vias 0 -> 1
- net /base_resistors/in: track 84.7 -> 154.1 mm
- net GND: track 32.7 -> 84.5 mm, vias 0 -> 18
- net -45V: track 20.0 -> 64.8 mm, vias 0 -> 1
- net /measured transistor/base_supp: track 0.00 -> 40.9 mm
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Other:
- board text added: "+-15V"
- board text added: "+-45V"
- board text added: "+12"
- board text added: "+24"
- board text added: "-24"
- board text added: "40-500V"
- board text added: "Base Measuring"
- board text added: "Base Supply"
- board text added: "Collector Measuring"
- board text added: "Collector Supply"
- board text added: "Emitter"
- board text added: "GND"
- board text added: "Rev: 1.0"
