File: Bipolar_transistor_tester_1.0/Bipolar_transistor_tester_1.0.kicad_pcb (KiCad board)
At the start: 4 copper layers, 170 x 140 mm, 250 parts, among them IC1 OPA454, IC2 OPA454, IC3 OPA454, IC4 OPA454, IC5 OPA454, J1 KF2510_7pin, J10 DJ621-6.3, J11 DJ621-6.3, J12 KF2510_3pin, J13 KF2510_6pin, J14 KF2510_6pin, J15 KF2510_5pin, J16 KF2510_5pin, J17 KF2510_2pin, J18 KF2510_2pin, J19 KF2510_5pin, J2 KF2510_6pin, J20 KF2510_5pin, J21 KF2510_6pin, J22 KF2510_4pin, J23 KF2510_2pin, J24 KF2510_2pin, J25 DJ621-6.3, J26 DJ621-6.3, J27 DJ621-6.3, J28 DJ621-6.3, J29 DJ621-6.3, J3 DJ621-6.3, J4 DJ621-6.3, J5 DJ621-6.3, J6 DJ621-6.3, J7 DJ621-6.3, J8 DJ621-6.3, J9 DJ621-6.3, Q1 AO3400A, Q2 AO3401A, Q3 IRFR9024, Q4 IRF640, Q5 AO3400A, Q6 AO3401A, Q7 IRFR9024, Q8 IRF640, U1 CPC1977, U10 PVN012, U11 CPC1977, U12 CPC1977, U13 PVN012, U14 PVN012, U15 PVN012, U16 PVN012, U17 INA118, U18 ISO124P, U19 PVN012, U2 PVN012, U20 PVN012, U21 AD549, U22 CPC1977, U23 PVG612, U24 PVN012, U25 OP07, U26 PVN012, U27 PVN012, U28 PVN012, U29 PVN012, U3 AD822, U30 PVN012, U31 CPC1977, U32 PVG612, U33 PVG612, U34 CPC1977, U35 AD822, U36 PVN012, U37 PVN012, U38 PVN012, U39 PVN012, U4 PVN012, U40 PVN012, U41 PVN012, U42 PVN012, U43 PVG612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

Commit message: bipolar tester add connectors numbers
Other:
- board text added: "1"
- board text added: "2"
- board text added: "3"
- board text added: "4"
- board text added: "5"
- board text added: "6"
- board text added: "7"
- board text added: "8"

Commit message: edit resistors cpc1977
Parts:
- Q4, Q8: value IRF640 -> IRFR4105
- renumbered U25 to U24, U24 to U25
