File: Bipolar_transistor_tester_1.0/base_cur_meter.sch (KiCad schematic (older format))
At the start: 10 parts, among them U8 INA118

Commit message: tester up
Parts:
- removed D11, D12, D13: PVN012, Package_DIP:DIP-6_W7.62mm, symbol Relay_SolidState:PVN012
- added C30, C31: 100n, Capacitor_SMD:C_0805_2012Metric, symbol Device:C
- added R76: 5 1%, Resistor_SMD:R_0805_2012Metric, symbol Device:R
- added R? (x4): 1k 1%, Resistor_SMD:R_0805_2012Metric, symbol Device:R
- added U44, U45, U46, U47: PVG612, Package_DIP:DIP-6_W7.62mm, symbol Relay_SolidState:PVG612
- C32: renamed from C4; value 100p -> 100n
- R74: renamed from R20; value 1M 1% -> 100k 1%
- R75: renamed from R21; value 10k 1% -> 1k 1%
- U48: renamed from U8; footprint (none) -> Package_DIP:DIP-8_W7.62mm
- renumbered R19 to R73, R22 to R77, R23 to R78
Connections:
- net +15V: now also C31.1
- net -15V: now also C30.1
- net GND: now also C30.2, C31.2
- net in+: now also R76.2
- net in-: now also U44.4, U45.4, U46.4, U47.4
- net at R74.1: now also U45.6
- net at R73.1: now also U44.6
- net at R75.1: now also U46.6
- net at R78.1, U48.6: no longer C32.1
- net ADC renamed adc3
- net adc3: now also C32.1
- new net: R?.2, U44.1
- new net: R?.2, U45.1
- new net: R?.2, U46.1
- new net: R?.2, U47.1
- new net: R76.1, U47.6
- new net 5_bcm1: U44.2
- new net 5_bcm2: U45.2
- new net 5_bcm3: U46.2
- new net 5_bcm4: U47.2
- new net 5_com_an: R?.1, R?.1, R?.1, R?.1
- no-connect marks 3 -> 4
Other:
- moved on the sheet: C32, R73, R74, R75, R78

Commit message: tester up
Parts:
- R99: renamed from R76; value 5 1% -> 5 1% 0.5W; footprint Resistor_SMD:R_0805_2012Metric -> Resistor_THT:R_Axial_DIN0309_L9.0mm_D3.2mm_P12.70mm_Horizontal
- gave numbers to parts that had none: 4
- renumbered R77 to R101, R78 to R102, R73 to R93, R74 to R95, R75 to R97
Other:
- moved on the sheet: R101
Changed lines of the file:
@@
 Sheet 10 11
 Title ""
-Date ""
+Date "2022-04-25"
 Rev ""
 Comp ""
@@
 $EndDescr
 $Comp
-L Device:R R74
+L Device:R R95
 U 1 1 6267BAA4
 P 4000 3500
-F 0 "R74" H 3950 3475 50  0000 R CNN
+F 0 "R95" H 3950 3475 50  0000 R CNN
 F 1 "100k 1%" H 3950 3550 50  0000 R CNN
 F 2 "Resistor_SMD:R_0805_2012Metric" V 3930 3500 50  0001 C CNN
@@
 $EndComp
 $Comp
-L Device:R R73
+L Device:R R93
 U 1 1 6267D1FF
 P 3250 3500
-F 0 "R73" H 3200 3475 50  0000 R CNN
+F 0 "R93" H 3200 3475 50  0000 R CNN
 F 1 "10M 1%" H 3200 3550 50  0000 R CNN
 F 2 "Resistor_SMD:R_0805_2012Metric" V 3180 3500 50  0001 C CNN
@@
 	3250 3800 3250 3650
 $Comp
-L Device:R R75
+L Device:R R97
 U 1 1 6275C9C8
 P 4800 3500
-F 0 "R75" H 4750 3475 50  0000 R CNN
+F 0 "R97" H 4750 3475 50  0000 R CNN
 F 1 "1k 1%" H 4750 3550 50  0000 R CNN
 F 2 "Resistor_SMD:R_0805_2012Metric" V 4730 3500 50  0001 C CNN
@@
 $EndComp
 $Comp
-L Device:R R78
+L Device:R R102
 U 1 1 62760733
 P 7550 3550
-F 0 "R78" V 7750 3600 50  0000 R CNN
+F 0 "R102" V 7750 3600 50  0000 R CNN
 F 1 "100" V 7650 3600 50  0000 R CNN
 F 2 "Resistor_SMD:R_0805_2012Metric" V 7480 3550 50  0001 C CNN
@@
 $EndComp
 $Comp
-L power:GND #PWR0122
+L power:GND #PWR0135
 U 1 1 62761C63
 P 7050 3950
-F 0 "#PWR0122" H 7050 3700 50  0001 C CNN
+F 0 "#PWR0135" H 7050 3700 50  0001 C CNN
 F 1 "GND" H 7055 3777 50  0000 C CNN
 F 2 "" H 7050 3950 50  0001 C CNN
@@
 $EndComp
 $Comp
-L power:-15V #PWR0121
+L power:-15V #PWR0134
 U 1 1 627626EF
 P 6800 3950
-F 0 "#PWR0121" H 6800 4050 50  0001 C CNN
+F 0 "#PWR0134" H 6800 4050 50  0001 C CNN
 F 1 "-15V" H 6815 4123 50  0000 C CNN
 F 2 "" H 6800 3950 50  0001 C CNN
@@
 	6800 3950 6800 3850
 $Comp
-L power:+15V #PWR0120
+L power:+15V #PWR0133
 U 1 1 6276323F
 P 6800 3150
-F 0 "#PWR0120" H 6800 3000 50  0001 C CNN
+F 0 "#PWR0133" H 6800 3000 50  0001 C CNN
 F 1 "+15V" H 6815 3323 50  0000 C CNN
 F 2 "" H 6800 3150 50  0001 C CNN
@@
 	6900 3950 6900 3850
 $Comp
-L power:GND #PWR0123
+L power:GND #PWR0136
 U 1 1 62764A89
 P 7900 4050
-F 0 "#PWR0123" H 7900 3800 50  0001 C CNN
+F 0 "#PWR0136" H 7900 3800 50  0001 C CNN
 F 1 "GND" H 7905 3877 50  0000 C CNN
 F 2 "" H 7900 4050 50  0001 C CNN
@@
 Connection ~ 4800 3350
 $Comp
-L Device:R R77
+L Device:R R101
 U 1 1 6276E3EC
-P 6300 3550
-F 0 "R77" H 6550 3500 50  0000 R CNN
-F 1 "51k 1%" H 6650 3600 50  0000 R CNN
-F 2 "Resistor_SMD:R_0805_2012Metric" V 6230 3550 50  0001 C CNN
-F 3 "~" H 6300 3550 50  0001 C CNN
-	1    6300 3550
+P 6400 3550
+F 0 "R101" H 6650 3500 50  0000 R CNN
+F 1 "51k 1%" H 6750 3600 50  0000 R CNN
+F 2 "Resistor_SMD:R_0805_2012Metric" V 6330 3550 50  0001 C CNN
+F 3 "~" H 6400 3550 50  0001 C CNN
+	1    6400 3550
 	-1   0    0    1
 $EndComp
@@
 Connection ~ 5000 3750
 Wire Wire Line
-	6300 3700 6500 3700
+	6400 3700 6500 3700
 Wire Wire Line
 	6500 3700 6500 3650
@@
 	6500 3450 6500 3400
 Wire Wire Line
-	6500 3400 6300 3400
+	6500 3400 6400 3400
 Wire Wire Line
 	7900 3700 7900 3550
@@
 Connection ~ 5800 3750
 $Comp
-L Device:R R76
+L Device:R R99
 U 1 1 626656EB
 P 5600 3500
-F 0 "R76" H 5550 3475 50  0000 R CNN
-F 1 "5 1%" H 5550 3550 50  0000 R CNN
-F 2 "Resistor_SMD:R_0805_2012Metric" V 5530 3500 50  0001 C CNN
+F 0 "R99" H 5550 3450 50  0000 R CNN
+F 1 "5 1% 0.5W" H 5550 3550 50  0000 R CNN
+F 2 "Resistor_THT:R_Axial_DIN0309_L9.0mm_D3.2mm_P12.70mm_Horizontal" V 5530 3500 50  0001 C CNN
 F 3 "~" H 5600 3500 50  0001 C CNN
 	1    5600 3500
@@
 AR Path="/62558810/62AD9041" Ref="#PWR?"  Part="1"
 AR Path="/62558C62/62AD9041" Ref="#PWR?"  Part="1"
-AR Path="/625CBDE7/62AD9041" Ref="#PWR0117"  Part="1"
-F 0 "#PWR0117" H 1650 5400 50  0001 C CNN
+AR Path="/625CBDE7/62AD9041" Ref="#PWR0130"  Part="1"
+F 0 "#PWR0130" H 1650 5400 50  0001 C CNN
 F 1 "-15V" H 1665 5473 50  0000 C CNN
 F 2 "" H 1650 5300 50  0001 C CNN
@@
 AR Path="/62558810/62AD9047" Ref="#PWR?"  Part="1"
 AR Path="/62558C62/62AD9047" Ref="#PWR?"  Part="1"
-AR Path="/625CBDE7/62AD9047" Ref="#PWR0119"  Part="1"
-F 0 "#PWR0119" H 2100 5150 50  0001 C CNN
+AR Path="/625CBDE7/62AD9047" Ref="#PWR0132"  Part="1"
+F 0 "#PWR0132" H 2100 5150 50  0001 C CNN
 F 1 "+15V" H 2115 5473 50  0000 C CNN
 F 2 "" H 2100 5300 50  0001 C CNN
@@
 AR Path="/62558810/62AD9050" Ref="#PWR?"  Part="1"
 AR Path="/62558C62/62AD9050" Ref="#PWR?"  Part="1"
-AR Path="/625CBDE7/62AD9050" Ref="#PWR0118"  Part="1"
-F 0 "#PWR0118" H 1900 5600 50  0001 C CNN
+AR Path="/625CBDE7/62AD9050" Ref="#PWR0131"  Part="1"
+F 0 "#PWR0131" H 1900 5600 50  0001 C CNN
 F 1 "GND" H 1905 5677 50  0000 C CNN
 F 2 "" H 1900 5850 50  0001 C CNN
@@
 5_com_an
 $Comp
-L Device:R R?
+L Device:R R94
 U 1 1 627EB650
 P 3250 4650
-F 0 "R?" H 3200 4625 50  0000 R CNN
+F 0 "R94" H 3200 4625 50  0000 R CNN
 F 1 "1k 1%" H 3200 4700 50  0000 R CNN
 F 2 "Resistor_SMD:R_0805_2012Metric" V 3180 4650 50  0001 C CNN
@@
 	3250 4500 3250 4400
 $Comp
-L Device:R R?
+L Device:R R96
 U 1 1 627EC490
 P 4000 4650
-F 0 "R?" H 3950 4625 50  0000 R CNN
+F 0 "R96" H 3950 4625 50  0000 R CNN
 F 1 "1k 1%" H 3950 4700 50  0000 R CNN
 F 2 "Resistor_SMD:R_0805_2012Metric" V 3930 4650 50  0001 C CNN
@@
 $EndComp
 $Comp
-L Device:R R?
+L Device:R R98
 U 1 1 627ECC29
 P 4800 4650
-F 0 "R?" H 4750 4625 50  0000 R CNN
+F 0 "R98" H 4750 4625 50  0000 R CNN
 F 1 "1k 1%" H 4750 4700 50  0000 R CNN
 F 2 "Resistor_SMD:R_0805_2012Metric" V 4730 4650 50  0001 C CNN
@@
 $EndComp
 $Comp
-L Device:R R?
+L Device:R R100
 U 1 1 627ED767
 P 5600 4650
-F 0 "R?" H 5550 4625 50  0000 R CNN
+F 0 "R100" H 5550 4625 50  0000 R CNN
 F 1 "1k 1%" H 5550 4700 50  0000 R CNN
 F 2 "Resistor_SMD:R_0805_2012Metric" V 5530 4650 50  0001 C CNN
