File: Bipolar_transistor_tester_1.0/base_resisrors.sch (KiCad schematic (older format))
At the start: 9 parts

Commit message: tester up
Parts:
- added R? (x5): 1k 1%, Resistor_SMD:R_0805_2012Metric, symbol Device:R
- R39: renamed from R10; value 1 -> 1 1%
- R40: renamed from R11; value 10 -> 10 1%
- R41: renamed from R12; value 100 -> 100 1%
- R42: renamed from R13; value 1k -> 1k 1%
- renumbered D5 to U26, D6 to U27, D7 to U28, D8 to U29, D9 to U30
Connections:
- net at U26.1: now also R?.1
- net 7_br1: now reaches U26.2
- net at U27.1: now also R?.1
- net 7_br2: now reaches U27.2
- net at U28.1: now also R?.1
- net 7_br3: now reaches U28.2
- net at U29.1: now also R?.1
- net 7_br4: now reaches U29.2
- net at U30.1: now also R?.1
- net 7_br5: now reaches U30.2
- net GND renamed gnd
- new net 7_com_an: R?.2, R?.2, R?.2, R?.2, R?.2
Other:
- moved on the sheet: U30
Changed lines of the file:
@@
 $Descr A4 11693 8268
 encoding utf-8
-Sheet 8 11
+Sheet 7 11
 Title ""
 Date ""
@@
 $EndDescr
 $Comp
-L Device:R R13
+L Device:R R42
 U 1 1 6269F7AC
 P 8450 2700
-F 0 "R13" H 8520 2746 50  0000 L CNN
-F 1 "1k" H 8520 2655 50  0000 L CNN
+F 0 "R42" H 8520 2746 50  0000 L CNN
+F 1 "1k 1%" H 8520 2655 50  0000 L CNN
 F 2 "Resistor_SMD:R_0805_2012Metric" V 8380 2700 50  0001 C CNN
 F 3 "~" H 8450 2700 50  0001 C CNN
@@
 $EndComp
 $Comp
-L Device:R R11
+L Device:R R40
 U 1 1 626A1674
 P 6000 2700
-F 0 "R11" H 6070 2746 50  0000 L CNN
-F 1 "10" H 6070 2655 50  0000 L CNN
+F 0 "R40" H 6070 2746 50  0000 L CNN
+F 1 "10 1%" H 6070 2655 50  0000 L CNN
 F 2 "Resistor_SMD:R_0805_2012Metric" V 5930 2700 50  0001 C CNN
 F 3 "~" H 6000 2700 50  0001 C CNN
@@
 $EndComp
 Connection ~ 6000 2550
-$Comp
-L power:GND #PWR0113
-U 1 1 626A5B64
-P 3300 3000
-F 0 "#PWR0113" H 3300 2750 50  0001 C CNN
-F 1 "GND" H 3305 2827 50  0000 C CNN
-F 2 "" H 3300 3000 50  0001 C CNN
-F 3 "" H 3300 3000 50  0001 C CNN
-	1    3300 3000
-	1    0    0    -1
-$EndComp
 Text HLabel 3300 2550 0    50   Input ~ 0
 in
 $Comp
-L Device:R R10
+L Device:R R39
 U 1 1 62724E56
 P 4800 2700
-F 0 "R10" H 4870 2746 50  0000 L CNN
-F 1 "1" H 4870 2655 50  0000 L CNN
+F 0 "R39" H 4870 2746 50  0000 L CNN
+F 1 "1 1%" H 4870 2655 50  0000 L CNN
 F 2 "Resistor_SMD:R_0805_2012Metric" V 4730 2700 50  0001 C CNN
 F 3 "~" H 4800 2700 50  0001 C CNN
@@
 	6000 2550 7250 2550
 $Comp
-L Device:R R12
+L Device:R R41
 U 1 1 62734339
 P 7250 2700
-F 0 "R12" H 7320 2746 50  0000 L CNN
-F 1 "100" H 7320 2655 50  0000 L CNN
+F 0 "R41" H 7320 2746 50  0000 L CNN
+F 1 "100 1%" H 7320 2655 50  0000 L CNN
 F 2 "Resistor_SMD:R_0805_2012Metric" V 7180 2700 50  0001 C CNN
 F 3 "~" H 7250 2700 50  0001 C CNN
@@
 	3300 2550 3750 2550
 $Comp
-L Relay_SolidState:PVN012 D5
+L Relay_SolidState:PVN012 U26
 U 1 1 62778BC0
 P 3850 3600
-F 0 "D5" V 3896 3420 50  0000 R CNN
+F 0 "U26" V 3896 3420 50  0000 R CNN
 F 1 "PVN012" V 3805 3420 50  0000 R CNN
 F 2 "Package_DIP:DIP-6_W7.62mm" H 3870 3800 50  0001 C CNN
@@
 $EndComp
 $Comp
-L Relay_SolidState:PVN012 D6
+L Relay_SolidState:PVN012 U27
 U 1 1 6277E396
 P 4900 3600
-F 0 "D6" V 4946 3420 50  0000 R CNN
+F 0 "U27" V 4946 3420 50  0000 R CNN
 F 1 "PVN012" V 4855 3420 50  0000 R CNN
 F 2 "Package_DIP:DIP-6_W7.62mm" H 4920 3800 50  0001 C CNN
@@
 $EndComp
 $Comp
-L Relay_SolidState:PVN012 D7
+L Relay_SolidState:PVN012 U28
 U 1 1 6277F3DA
 P 6100 3600
-F 0 "D7" V 6146 3420 50  0000 R CNN
+F 0 "U28" V 6146 3420 50  0000 R CNN
 F 1 "PVN012" V 6055 3420 50  0000 R CNN
 F 2 "Package_DIP:DIP-6_W7.62mm" H 6120 3800 50  0001 C CNN
@@
 $EndComp
 $Comp
-L Relay_SolidState:PVN012 D8
+L Relay_SolidState:PVN012 U29
 U 1 1 62780068
 P 7350 3550
-F 0 "D8" V 7396 3370 50  0000 R CNN
+F 0 "U29" V 7396 3370 50  0000 R CNN
 F 1 "PVN012" V 7305 3370 50  0000 R CNN
 F 2 "Package_DIP:DIP-6_W7.62mm" H 7370 3750 50  0001 C CNN
@@
 $EndComp
 $Comp
-L Relay_SolidState:PVN012 D9
+L Relay_SolidState:PVN012 U30
 U 1 1 62781063
-P 8550 3500
-F 0 "D9" V 8596 3320 50  0000 R CNN
-F 1 "PVN012" V 8505 3320 50  0000 R CNN
-F 2 "Package_DIP:DIP-6_W7.62mm" H 8570 3700 50  0001 C CNN
-F 3 "" H 8570 3700 50  0001 C CNN
-	1    8550 3500
-	0    -1   -1   0
-$EndComp
-Wire Wire Line
-	8650 3200 8650 3000
-Wire Wire Line
-	8450 3200 8450 2850
+P 8550 3550
+F 0 "U30" V 8596 3370 50  0000 R CNN
+F 1 "PVN012" V 8505 3370 50  0000 R CNN
+F 2 "Package_DIP:DIP-6_W7.62mm" H 8570 3750 50  0001 C CNN
+F 3 "" H 8570 3750 50  0001 C CNN
+	1    8550 3550
+	0    -1   -1   0
+$EndComp
 Wire Wire Line
 	7450 3250 7450 3000
@@
 NoConn ~ 6100 3300
 NoConn ~ 7350 3250
-NoConn ~ 8550 3200
+NoConn ~ 8550 3250
+Text HLabel 3300 3000 0    50   Input ~ 0
+gnd
+Text GLabel 3600 4350 0    50   Input ~ 0
+7_com_an
+$Comp
+L Device:R R?
+U 1 1 6281361E
+P 3750 4200
+F 0 "R?" H 3820 4246 50  0000 L CNN
+F 1 "1k 1%" H 3820 4155 50  0000 L CNN
+F 2 "Resistor_SMD:R_0805_2012Metric" V 3680 4200 50  0001 C CNN
+F 3 "~" H 3750 4200 50  0001 C CNN
+	1    3750 4200
+	1    0    0    -1
+$EndComp
+Wire Wire Line
+	3750 4350 3600 4350
+Wire Wire Line
+	3750 3900 3750 4050
+Text GLabel 4650 4350 0    50   Input ~ 0
+7_com_an
+$Comp
+L Device:R R?
+U 1 1 628155FF
+P 4800 4200
+F 0 "R?" H 4870 4246 50  0000 L CNN
+F 1 "1k 1%" H 4870 4155 50  0000 L CNN
+F 2 "Resistor_SMD:R_0805_2012Metric" V 4730 4200 50  0001 C CNN
+F 3 "~" H 4800 4200 50  0001 C CNN
+	1    4800 4200
+	1    0    0    -1
+$EndComp
+Wire Wire Line
+	4800 4350 4650 4350
+Wire Wire Line
+	4800 3900 4800 4050
+Text GLabel 5850 4350 0    50   Input ~ 0
+7_com_an
+$Comp
+L Device:R R?
+U 1 1 62815E01
+P 6000 4200
+F 0 "R?" H 6070 4246 50  0000 L CNN
+F 1 "1k 1%" H 6070 4155 50  0000 L CNN
+F 2 "Resistor_SMD:R_0805_2012Metric" V 5930 4200 50  0001 C CNN
+F 3 "~" H 6000 4200 50  0001 C CNN
+	1    6000 4200
+	1    0    0    -1
+$EndComp
+Wire Wire Line
+	6000 4350 5850 4350
+Wire Wire Line
+	6000 3900 6000 4050
+Text GLabel 7100 4300 0    50   Input ~ 0
+7_com_an
+$Comp
+L Device:R R?
+U 1 1 6281651F
+P 7250 4150
+F 0 "R?" H 7320 4196 50  0000 L CNN
+F 1 "1k 1%" H 7320 4105 50  0000 L CNN
+F 2 "Resistor_SMD:R_0805_2012Metric" V 7180 4150 50  0001 C CNN
+F 3 "~" H 7250 4150 50  0001 C CNN
+	1    7250 4150
+	1    0    0    -1
+$EndComp
+Wire Wire Line
+	7250 4300 7100 4300
+Wire Wire Line
+	7250 3850 7250 4000
+Text GLabel 8300 4300 0    50   Input ~ 0
+7_com_an
+$Comp
+L Device:R R?
+U 1 1 62816D2F
+P 8450 4150
+F 0 "R?" H 8520 4196 50  0000 L CNN
+F 1 "1k 1%" H 8520 4105 50  0000 L CNN
+F 2 "Resistor_SMD:R_0805_2012Metric" V 8380 4150 50  0001 C CNN
+F 3 "~" H 8450 4150 50  0001 C CNN
+	1    8450 4150
+	1    0    0    -1
+$EndComp
+Wire Wire Line
+	8450 4300 8300 4300
+Text GLabel 4050 4000 2    50   Input ~ 0
+7_br1
+Wire Wire Line
+	4050 4000 3950 4000
+Wire Wire Line
+	3950 4000 3950 3900
+Text GLabel 5100 4000 2    50   Input ~ 0
+7_br2
+Text GLabel 6300 4000 2    50   Input ~ 0
+7_br3
+Text GLabel 7550 3950 2    50   Input ~ 0
+7_br4
+Text GLabel 8750 3950 2    50   Input ~ 0
+7_br5
+Wire Wire Line
+	8750 3950 8650 3950
+Wire Wire Line
+	8650 3950 8650 3850
+Wire Wire Line
+	7550 3950 7450 3950
+Wire Wire Line
+	7450 3950 7450 3850
+Wire Wire Line
+	6300 4000 6200 4000
+Wire Wire Line
+	6200 4000 6200 3900
+Wire Wire Line
+	5100 4000 5000 4000
+Wire Wire Line
+	5000 4000 5000 3900
+Wire Wire Line
+	8450 2850 8450 3250
+Wire Wire Line
+	8650 3000 8650 3250
+Wire Wire Line
+	8450 4000 8450 3850
 $EndSCHEMATC

Commit message: tester up
Parts:
- gave numbers to parts that had none: 5
- renumbered R39 to R51, R40 to R53, R41 to R55, R42 to R57
Changed lines of the file:
@@
 Sheet 7 11
 Title ""
-Date ""
+Date "2022-04-25"
 Rev ""
 Comp ""
@@
 $EndDescr
 $Comp
-L Device:R R42
+L Device:R R57
 U 1 1 6269F7AC
 P 8450 2700
-F 0 "R42" H 8520 2746 50  0000 L CNN
+F 0 "R57" H 8520 2746 50  0000 L CNN
 F 1 "1k 1%" H 8520 2655 50  0000 L CNN
 F 2 "Resistor_SMD:R_0805_2012Metric" V 8380 2700 50  0001 C CNN
@@
 $EndComp
 $Comp
-L Device:R R40
+L Device:R R53
 U 1 1 626A1674
 P 6000 2700
-F 0 "R40" H 6070 2746 50  0000 L CNN
+F 0 "R53" H 6070 2746 50  0000 L CNN
 F 1 "10 1%" H 6070 2655 50  0000 L CNN
 F 2 "Resistor_SMD:R_0805_2012Metric" V 5930 2700 50  0001 C CNN
@@
 in
 $Comp
-L Device:R R39
+L Device:R R51
 U 1 1 62724E56
 P 4800 2700
-F 0 "R39" H 4870 2746 50  0000 L CNN
+F 0 "R51" H 4870 2746 50  0000 L CNN
 F 1 "1 1%" H 4870 2655 50  0000 L CNN
 F 2 "Resistor_SMD:R_0805_2012Metric" V 4730 2700 50  0001 C CNN
@@
 	6000 2550 7250 2550
 $Comp
-L Device:R R41
+L Device:R R55
 U 1 1 62734339
 P 7250 2700
-F 0 "R41" H 7320 2746 50  0000 L CNN
+F 0 "R55" H 7320 2746 50  0000 L CNN
 F 1 "100 1%" H 7320 2655 50  0000 L CNN
 F 2 "Resistor_SMD:R_0805_2012Metric" V 7180 2700 50  0001 C CNN
@@
 7_com_an
 $Comp
-L Device:R R?
+L Device:R R50
 U 1 1 6281361E
 P 3750 4200
-F 0 "R?" H 3820 4246 50  0000 L CNN
+F 0 "R50" H 3820 4246 50  0000 L CNN
 F 1 "1k 1%" H 3820 4155 50  0000 L CNN
 F 2 "Resistor_SMD:R_0805_2012Metric" V 3680 4200 50  0001 C CNN
@@
 7_com_an
 $Comp
-L Device:R R?
+L Device:R R52
 U 1 1 628155FF
 P 4800 4200
-F 0 "R?" H 4870 4246 50  0000 L CNN
+F 0 "R52" H 4870 4246 50  0000 L CNN
 F 1 "1k 1%" H 4870 4155 50  0000 L CNN
 F 2 "Resistor_SMD:R_0805_2012Metric" V 4730 4200 50  0001 C CNN
@@
 7_com_an
 $Comp
-L Device:R R?
+L Device:R R54
 U 1 1 62815E01
 P 6000 4200
-F 0 "R?" H 6070 4246 50  0000 L CNN
+F 0 "R54" H 6070 4246 50  0000 L CNN
 F 1 "1k 1%" H 6070 4155 50  0000 L CNN
 F 2 "Resistor_SMD:R_0805_2012Metric" V 5930 4200 50  0001 C CNN
@@
 7_com_an
 $Comp
-L Device:R R?
+L Device:R R56
 U 1 1 6281651F
 P 7250 4150
-F 0 "R?" H 7320 4196 50  0000 L CNN
+F 0 "R56" H 7320 4196 50  0000 L CNN
 F 1 "1k 1%" H 7320 4105 50  0000 L CNN
 F 2 "Resistor_SMD:R_0805_2012Metric" V 7180 4150 50  0001 C CNN
@@
 7_com_an
 $Comp
-L Device:R R?
+L Device:R R58
 U 1 1 62816D2F
 P 8450 4150
-F 0 "R?" H 8520 4196 50  0000 L CNN
+F 0 "R58" H 8520 4196 50  0000 L CNN
 F 1 "1k 1%" H 8520 4105 50  0000 L CNN
 F 2 "Resistor_SMD:R_0805_2012Metric" V 8380 4150 50  0001 C CNN
