File: Bipolar_transistor_tester_1.0/collector_сur_meter.sch (KiCad schematic (older format))
At the start: 16 parts, among them U1 INA118

Commit message: tester up
Parts:
- added C5, C6: 100n, Capacitor_SMD:C_0805_2012Metric, symbol Device:C
- added R? (x4): 1k 1%, Resistor_SMD:R_0805_2012Metric, symbol Device:R
- C9: renamed from C?; value 100p -> 100n
- R28: renamed from R?; value 1 1% -> 10 1%
- U17: renamed from U1; footprint (none) -> Package_DIP:DIP-8_W7.62mm
- gave numbers to parts that had none: 12
- renumbered R1 to R31
Connections:
- net +15V: now also C6.1
- net -15V: now also C5.1
- net GND: now also C5.2, C6.2
- net at U16.1: now also R?.1
- net 3_ccm4: now reaches U16.2
- net at U15.1: now also R?.1
- net 3_ccm3: now reaches U15.2
- net at U14.1: now also R?.1
- net 3_ccm2: now reaches U14.2
- net at U13.1: now also R?.1
- net 3_ccm1: now reaches U13.2
- net out renamed adc0
- new net 3_com_an: R?.2, R?.2, R?.2, R?.2
Other:
- moved on the sheet: C7, C8, C9, PS1, R27, R28, R29, R30, R31, R32, U13, U14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

Commit message: tester up
Parts:
- R29: renamed from R27; value 0,1 1% -> 0,1 1% 0.5W; footprint Resistor_SMD:R_0805_2012Metric -> Resistor_THT:R_Axial_DIN0309_L9.0mm_D3.2mm_P12.70mm_Horizontal
- R31: renamed from R28; value 10 1% -> 10 1% 0.5W; footprint Resistor_SMD:R_0805_2012Metric -> Resistor_THT:R_Axial_DIN0309_L9.0mm_D3.2mm_P12.70mm_Horizontal
- gave numbers to parts that had none: 4
- renumbered R29 to R33, R30 to R35, R31 to R37, R32 to R38
Changed lines of the file:
@@
 Sheet 3 11
 Title ""
-Date ""
+Date "2022-04-25"
 Rev ""
 Comp ""
@@
 $EndComp
 $Comp
-L Device:R R31
+L Device:R R37
 U 1 1 62656C18
 P 5600 2950
-F 0 "R31" H 5670 2996 50  0000 L CNN
+F 0 "R37" H 5670 2996 50  0000 L CNN
 F 1 "2k 1%" H 5670 2905 50  0000 L CNN
 F 2 "Resistor_SMD:R_0805_2012Metric" V 5530 2950 50  0001 C CNN
@@
 	8175 3425 8175 3275
 $Comp
-L Device:R R32
+L Device:R R38
 U 1 1 6264600A
 P 9350 2650
-F 0 "R32" V 9150 2600 50  0000 L CNN
+F 0 "R38" V 9150 2600 50  0000 L CNN
 F 1 "100" V 9250 2550 50  0000 L CNN
 F 2 "Resistor_SMD:R_0805_2012Metric" V 9280 2650 50  0001 C CNN
@@
 $EndComp
 $Comp
-L Device:R R30
+L Device:R R35
 U 1 1 62663172
 P 5050 3000
-F 0 "R30" H 5120 3046 50  0000 L CNN
+F 0 "R35" H 5120 3046 50  0000 L CNN
 F 1 "100k 1%" H 5120 2955 50  0000 L CNN
 F 2 "Resistor_SMD:R_0805_2012Metric" V 4980 3000 50  0001 C CNN
@@
 	5250 3300 4450 3300
 $Comp
-L Device:R R27
+L Device:R R29
 U 1 1 62676DF3
 P 2700 3000
-F 0 "R27" H 2770 3046 50  0000 L CNN
-F 1 "0,1 1%" H 2770 2955 50  0000 L CNN
-F 2 "Resistor_SMD:R_0805_2012Metric" V 2630 3000 50  0001 C CNN
+F 0 "R29" H 2770 3046 50  0000 L CNN
+F 1 "0,1 1% 0.5W" H 2770 2955 50  0000 L CNN
+F 2 "Resistor_THT:R_Axial_DIN0309_L9.0mm_D3.2mm_P12.70mm_Horizontal" V 2630 3000 50  0001 C CNN
 F 3 "~" H 2700 3000 50  0001 C CNN
 	1    2700 3000
@@
 	2700 3150 2700 3400
 $Comp
-L Device:R R28
+L Device:R R31
 U 1 1 6267C59A
 P 3500 3000
-F 0 "R28" H 3570 3046 50  0000 L CNN
-F 1 "10 1%" H 3570 2955 50  0000 L CNN
-F 2 "Resistor_SMD:R_0805_2012Metric" V 3430 3000 50  0001 C CNN
+F 0 "R31" H 3570 3046 50  0000 L CNN
+F 1 "10 1% 0.5W" H 3570 2955 50  0000 L CNN
+F 2 "Resistor_THT:R_Axial_DIN0309_L9.0mm_D3.2mm_P12.70mm_Horizontal" V 3430 3000 50  0001 C CNN
 F 3 "~" H 3500 3000 50  0001 C CNN
 	1    3500 3000
@@
 $EndComp
 $Comp
-L Device:R R29
+L Device:R R33
 U 1 1 6267CCE2
 P 4250 3000
-F 0 "R29" H 4320 3046 50  0000 L CNN
+F 0 "R33" H 4320 3046 50  0000 L CNN
 F 1 "1k 1%" H 4320 2955 50  0000 L CNN
 F 2 "Resistor_SMD:R_0805_2012Metric" V 4180 3000 50  0001 C CNN
@@
 	3400 5700 3150 5700
 $Comp
-L Device:R R?
+L Device:R R30
 U 1 1 627B2648
 P 2700 4250
-F 0 "R?" H 2770 4296 50  0000 L CNN
+F 0 "R30" H 2770 4296 50  0000 L CNN
 F 1 "1k 1%" H 2770 4205 50  0000 L CNN
 F 2 "Resistor_SMD:R_0805_2012Metric" V 2630 4250 50  0001 C CNN
@@
 $EndComp
 $Comp
-L Device:R R?
+L Device:R R32
 U 1 1 627B3165
 P 3500 4250
-F 0 "R?" H 3570 4296 50  0000 L CNN
+F 0 "R32" H 3570 4296 50  0000 L CNN
 F 1 "1k 1%" H 3570 4205 50  0000 L CNN
 F 2 "Resistor_SMD:R_0805_2012Metric" V 3430 4250 50  0001 C CNN
@@
 $EndComp
 $Comp
-L Device:R R?
+L Device:R R34
 U 1 1 627B34F0
 P 4250 4250
-F 0 "R?" H 4320 4296 50  0000 L CNN
+F 0 "R34" H 4320 4296 50  0000 L CNN
 F 1 "1k 1%" H 4320 4205 50  0000 L CNN
 F 2 "Resistor_SMD:R_0805_2012Metric" V 4180 4250 50  0001 C CNN
@@
 $EndComp
 $Comp
-L Device:R R?
+L Device:R R36
 U 1 1 627B36E3
 P 5050 4250
-F 0 "R?" H 5120 4296 50  0000 L CNN
+F 0 "R36" H 5120 4296 50  0000 L CNN
 F 1 "1k 1%" H 5120 4205 50  0000 L CNN
 F 2 "Resistor_SMD:R_0805_2012Metric" V 4980 4250 50  0001 C CNN

Commit message: tester up
Parts:
- added C33, C35, C36: 100n, Capacitor_SMD:C_0805_2012Metric, symbol Device:C
- added C34: 1u, Capacitor_SMD:C_0805_2012Metric, symbol Device:C
Connections:
- net +12V: now also C33.1, C34.1
- net GND: now also C33.2, C34.2
- net GND2: now also C35.2, C36.2
- net at C7.1, PS1.4 (-Vout), U17.4 (V-)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: now also C35.1
- net at C8.1, PS1.6 (+Vout), U17.7 (V+)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: now also C36.1
Other:
- moved on the sheet: R29, R30, R31, R32, R33, R34, R35, R36, U13, U14, U15, U16
