File: Bipolar_transistor_tester_1.0/connectors.sch (KiCad schematic (older format))
At the start: 32 parts, among them J1 KF2510_7pin, J10 DJ621-6.3, J11 DJ621-6.3, J2 KF2510_6pin, J3 DJ621-6.3, J4 DJ621-6.3, J5 DJ621-6.3, J6 DJ621-6.3, J7 DJ621-6.3, J8 DJ621-6.3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

Commit message: tester up
Parts:
- removed J? (x2): KF2510_2pin, Connector_KF2510:KF2510_2pin, symbol Connector:Conn_01x02_Male
- added J12: KF2510_3pin, Connector_KF2510:KF2510_3pin, symbol Connector:Conn_01x03_Male
- J10, J11, J3, J4, J5, J6, J7, J8, J9: footprint Connector:CONN_63824-1 -> Connector:Knife_Terminal_6.3mm_P5.00mm_Vertical
- gave numbers to parts that had none: 12
Connections:
- net +12C is gone; now on net +12V: J8.1 (Pin_1)
- net GND: now also J12.1 (Pin_1)
- net dac0: now also J12.2 (Pin_2)
- net dac1: now also J12.3 (Pin_3)
Other:
- moved on the sheet: J3
