File: Bipolar_transistor_tester_1.0/emitter_cur_meter.sch (KiCad schematic (older format))
At the start: 12 parts, among them U2 AD549

Commit message: tester up
Parts:
- removed D1: PVN012, Package_DIP:DIP-6_W7.62mm, symbol Relay_SolidState:PVN012
- removed R4: 100k 1%, Resistor_SMD:R_0805_2012Metric, symbol Device:R
- removed R5: 10M 1%, Resistor_SMD:R_0805_2012Metric, symbol Device:R
- added C17, C18: 100n, Capacitor_SMD:C_0805_2012Metric, symbol Device:C
- added R? (x2): 1k 1%, Resistor_SMD:R_0805_2012Metric, symbol Device:R
- C20: renamed from C2; value 100p -> 100n
- R34: renamed from R2; value 10M 1% -> 100M 1%
- RV1: value 10k -> PV32H103; footprint (none) -> Potentiometer_THT:Potentiometer_Bourns_3339H_Vertical
- renumbered C1 to C19, R3 to R33, R6 to R35, D2 to U19, D3 to U20, U2 to U21
Connections:
- net +15V: now also C18.1
- net -15V: now also C17.1
- net GND: now also C17.2, C18.2
- net at C19.2, R33.1, R35.2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: now also R34.1
- net at R33.2: now also U19.4; no longer U19.6
- net in: now reaches U20.6
- net in: now also C19.1, U19.6, U21.2 (-); no longer R34.1
- net at U20.1: now also R?.1
- net 4_ecm2: now reaches U20.2
- net at U20.4: now also R34.2
- net at U19.1: now also R?.1
- net 4_ecm1: now reaches U19.2
- net adc renamed adc1
- net in+ renamed gnd
- removed net in-: C19.1, R34.2, U19.4, U21.2 (-)
- new net 4_com_an: R?.2, R?.2
Other:
- moved on the sheet: C19, C20, R33, R34, R35, RV1, U19, U20, U21

Commit message: tester up
Parts:
- gave numbers to parts that had none: 2
- renumbered R33 to R41, R34 to R42, R35 to R43
Connections:
- net gnd renamed to_gnd
Changed lines of the file:
@@
 Sheet 5 11
 Title ""
-Date ""
+Date "2022-04-25"
 Rev ""
 Comp ""
@@
 $EndComp
 $Comp
-L Device:R R35
+L Device:R R43
 U 1 1 62792B87
 P 7200 2900
-F 0 "R35" V 6993 2900 50  0000 C CNN
+F 0 "R43" V 6993 2900 50  0000 C CNN
 F 1 "100" V 7084 2900 50  0000 C CNN
 F 2 "Resistor_SMD:R_0805_2012Metric" V 7130 2900 50  0001 C CNN
@@
 $EndComp
 $Comp
-L power:-15V #PWR072
+L power:-15V #PWR085
 U 1 1 62793C79
 P 6400 3300
-F 0 "#PWR072" H 6400 3400 50  0001 C CNN
+F 0 "#PWR085" H 6400 3400 50  0001 C CNN
 F 1 "-15V" H 6415 3473 50  0000 C CNN
 F 2 "" H 6400 3300 50  0001 C CNN
@@
 $EndComp
 $Comp
-L Device:R R33
+L Device:R R41
 U 1 1 62794B04
 P 6500 4500
-F 0 "R33" V 6293 4500 50  0000 C CNN
+F 0 "R41" V 6293 4500 50  0000 C CNN
 F 1 "1k 1%" V 6384 4500 50  0000 C CNN
 F 2 "Resistor_SMD:R_0805_2012Metric" V 6430 4500 50  0001 C CNN
@@
 $EndComp
 $Comp
-L Device:R R34
+L Device:R R42
 U 1 1 627953F9
 P 6500 5150
-F 0 "R34" V 6293 5150 50  0000 C CNN
+F 0 "R42" V 6293 5150 50  0000 C CNN
 F 1 "100M 1%" V 6384 5150 50  0000 C CNN
 F 2 "Resistor_SMD:R_0805_2012Metric" V 6430 5150 50  0001 C CNN
@@
 	6400 3300 6400 3200
 $Comp
-L power:+15V #PWR071
+L power:+15V #PWR084
 U 1 1 6279F4B4
 P 6400 2500
-F 0 "#PWR071" H 6400 2350 50  0001 C CNN
+F 0 "#PWR084" H 6400 2350 50  0001 C CNN
 F 1 "+15V" H 6415 2673 50  0000 C CNN
 F 2 "" H 6400 2500 50  0001 C CNN
@@
 	6400 2500 6400 2600
 Text HLabel 5250 2800 0    50   Input ~ 0
-gnd
+to_gnd
 Wire Wire Line
 	7350 2900 7550 2900
@@
 	7550 2900 7850 2900
 $Comp
-L power:GND #PWR074
+L power:GND #PWR087
 U 1 1 627A280C
 P 7550 3350
-F 0 "#PWR074" H 7550 3100 50  0001 C CNN
+F 0 "#PWR087" H 7550 3100 50  0001 C CNN
 F 1 "GND" H 7555 3177 50  0000 C CNN
 F 2 "" H 7550 3350 50  0001 C CNN
@@
 	6800 2900 6900 2900
 $Comp
-L power:-15V #PWR073
+L power:-15V #PWR086
 U 1 1 62650BB0
 P 7000 3600
-F 0 "#PWR073" H 7000 3700 50  0001 C CNN
+F 0 "#PWR086" H 7000 3700 50  0001 C CNN
 F 1 "-15V" H 7015 3773 50  0000 C CNN
 F 2 "" H 7000 3600 50  0001 C CNN
@@
 AR Path="/62558810/62ACEE50" Ref="#PWR?"  Part="1"
 AR Path="/62558C62/62ACEE50" Ref="#PWR?"  Part="1"
-AR Path="/62559320/62ACEE50" Ref="#PWR068"  Part="1"
-F 0 "#PWR068" H 2850 3650 50  0001 C CNN
+AR Path="/62559320/62ACEE50" Ref="#PWR081"  Part="1"
+F 0 "#PWR081" H 2850 3650 50  0001 C CNN
 F 1 "-15V" H 2865 3723 50  0000 C CNN
 F 2 "" H 2850 3550 50  0001 C CNN
@@
 AR Path="/62558810/62ACEE56" Ref="#PWR?"  Part="1"
 AR Path="/62558C62/62ACEE56" Ref="#PWR?"  Part="1"
-AR Path="/62559320/62ACEE56" Ref="#PWR070"  Part="1"
-F 0 "#PWR070" H 3300 3400 50  0001 C CNN
+AR Path="/62559320/62ACEE56" Ref="#PWR083"  Part="1"
+F 0 "#PWR083" H 3300 3400 50  0001 C CNN
 F 1 "+15V" H 3315 3723 50  0000 C CNN
 F 2 "" H 3300 3550 50  0001 C CNN
@@
 AR Path="/62558810/62ACEE5F" Ref="#PWR?"  Part="1"
 AR Path="/62558C62/62ACEE5F" Ref="#PWR?"  Part="1"
-AR Path="/62559320/62ACEE5F" Ref="#PWR069"  Part="1"
-F 0 "#PWR069" H 3100 3850 50  0001 C CNN
+AR Path="/62559320/62ACEE5F" Ref="#PWR082"  Part="1"
+F 0 "#PWR082" H 3100 3850 50  0001 C CNN
 F 1 "GND" H 3105 3927 50  0000 C CNN
 F 2 "" H 3100 4100 50  0001 C CNN
@@
 4_com_an
 $Comp
-L Device:R R?
+L Device:R R39
 U 1 1 627DAEA8
 P 5050 4300
-F 0 "R?" V 4843 4300 50  0000 C CNN
+F 0 "R39" V 4843 4300 50  0000 C CNN
 F 1 "1k 1%" V 4934 4300 50  0000 C CNN
 F 2 "Resistor_SMD:R_0805_2012Metric" V 4980 4300 50  0001 C CNN
@@
 4_com_an
 $Comp
-L Device:R R?
+L Device:R R40
 U 1 1 627DCF4C
 P 5050 4950
-F 0 "R?" V 4843 4950 50  0000 C CNN
+F 0 "R40" V 4843 4950 50  0000 C CNN
 F 1 "1k 1%" V 4934 4950 50  0000 C CNN
 F 2 "Resistor_SMD:R_0805_2012Metric" V 4980 4950 50  0001 C CNN
