File: Bipolar_transistor_tester_1.0/transistor.sch (KiCad schematic (older format))
At the start: 6 parts, among them J1 DJ621-6.3, J2 DJ621-6.3, J3 DJ621-6.3, J4 DJ621-6.3, J5 DJ621-6.3, J6 DJ621-6.3

Commit message: tester up
Parts:
- removed J1, J2, J3, J4, J5, J6: DJ621-6.3, symbol Connector:Conn_01x01_Male
- added J12, J13, J14, J15, J16: DJ621-6.3, Connector:CONN_63824-1, symbol Connector:Conn_01x01_Male
Connections:
- net base_meas: now also J15.1 (Pin_1)
- net base_supp: now also J14.1 (Pin_1)
- net coll_meas: now also J13.1 (Pin_1)
- net coll_supp: now also J12.1 (Pin_1)
- new net emitter: J16.1 (Pin_1)
Changed lines of the file:
@@
 $Descr A4 11693 8268
 encoding utf-8
-Sheet 2 11
+Sheet 11 11
 Title ""
 Date ""
@@
 Comment4 ""
 $EndDescr
-$Comp
-L Connector:Conn_01x01_Male J3
-U 1 1 6253E64D
-P 5275 4050
-F 0 "J3" H 5383 4231 50  0000 C CNN
-F 1 "DJ621-6.3" H 5383 4140 50  0000 C CNN
-F 2 "" H 5275 4050 50  0001 C CNN
-F 3 "~" H 5275 4050 50  0001 C CNN
-	1    5275 4050
-	1    0    0    -1
-$EndComp
-$Comp
-L Connector:Conn_01x01_Male J2
-U 1 1 6254A083
-P 5275 3750
-F 0 "J2" H 5383 3931 50  0000 C CNN
-F 1 "DJ621-6.3" H 5383 3840 50  0000 C CNN
-F 2 "" H 5275 3750 50  0001 C CNN
-F 3 "~" H 5275 3750 50  0001 C CNN
-	1    5275 3750
-	1    0    0    -1
-$EndComp
-$Comp
-L Connector:Conn_01x01_Male J1
-U 1 1 6254A777
-P 5275 2150
-F 0 "J1" H 5383 2331 50  0000 C CNN
-F 1 "DJ621-6.3" H 5383 2240 50  0000 C CNN
-F 2 "" H 5275 2150 50  0001 C CNN
-F 3 "~" H 5275 2150 50  0001 C CNN
-	1    5275 2150
-	1    0    0    -1
-$EndComp
-$Comp
-L Connector:Conn_01x01_Male J6
-U 1 1 6254BD3A
-P 5300 2450
-F 0 "J6" H 5408 2631 50  0000 C CNN
-F 1 "DJ621-6.3" H 5408 2540 50  0000 C CNN
-F 2 "" H 5300 2450 50  0001 C CNN
-F 3 "~" H 5300 2450 50  0001 C CNN
-	1    5300 2450
-	1    0    0    -1
-$EndComp
-$Comp
-L Connector:Conn_01x01_Male J5
-U 1 1 6254BFBD
-P 5275 5800
-F 0 "J5" H 5383 5981 50  0000 C CNN
-F 1 "DJ621-6.3" H 5383 5890 50  0000 C CNN
-F 2 "" H 5275 5800 50  0001 C CNN
-F 3 "~" H 5275 5800 50  0001 C CNN
-	1    5275 5800
-	1    0    0    -1
-$EndComp
-$Comp
-L Connector:Conn_01x01_Male J4
-U 1 1 6254C63E
-P 5275 5500
-F 0 "J4" H 5383 5681 50  0000 C CNN
-F 1 "DJ621-6.3" H 5383 5590 50  0000 C CNN
-F 2 "" H 5275 5500 50  0001 C CNN
-F 3 "~" H 5275 5500 50  0001 C CNN
-	1    5275 5500
-	1    0    0    -1
-$EndComp
 Text HLabel 6300 2150 2    50   Input ~ 0
 coll_supp
@@
 Text HLabel 6225 3750 2    50   Input ~ 0
 base_supp
-Text HLabel 6100 5800 2    50   Input ~ 0
-emit_meas
 Text HLabel 6100 5500 2    50   Input ~ 0
-emit_supp
+emitter
 Wire Wire Line
-	6100 5500 5475 5500
+	6100 5500 5500 5500
 Wire Wire Line
-	6100 5800 5475 5800
+	6225 3750 5500 3750
 Wire Wire Line
-	6225 3750 5475 3750
+	6250 4050 5500 4050
 Wire Wire Line
-	6250 4050 5475 4050
-Wire Wire Line
-	6300 2150 5475 2150
+	6300 2150 5500 2150
 Text HLabel 6275 2450 2    50   Input ~ 0
 coll_meas
 Wire Wire Line
 	6275 2450 5500 2450
+$Comp
+L Connector:Conn_01x01_Male J12
+U 1 1 62AE5BCB
+P 5300 2150
+F 0 "J12" H 5408 2331 50  0000 C CNN
+F 1 "DJ621-6.3" H 5408 2240 50  0000 C CNN
+F 2 "Connector:CONN_63824-1" H 5300 2150 50  0001 C CNN
+F 3 "~" H 5300 2150 50  0001 C CNN
+	1    5300 2150
+	1    0    0    -1
+$EndComp
+$Comp
+L Connector:Conn_01x01_Male J14
+U 1 1 62AE5F58
+P 5300 3750
+F 0 "J14" H 5408 3931 50  0000 C CNN
+F 1 "DJ621-6.3" H 5408 3840 50  0000 C CNN
+F 2 "Connector:CONN_63824-1" H 5300 3750 50  0001 C CNN
+F 3 "~" H 5300 3750 50  0001 C CNN
+	1    5300 3750
+	1    0    0    -1
+$EndComp
+$Comp
+L Connector:Conn_01x01_Male J15
+U 1 1 62AE6B77
+P 5300 4050
+F 0 "J15" H 5408 4231 50  0000 C CNN
+F 1 "DJ621-6.3" H 5408 4140 50  0000 C CNN
+F 2 "Connector:CONN_63824-1" H 5300 4050 50  0001 C CNN
+F 3 "~" H 5300 4050 50  0001 C CNN
+	1    5300 4050
+	1    0    0    -1
+$EndComp
+$Comp
+L Connector:Conn_01x01_Male J16
+U 1 1 62AE7081
+P 5300 5500
+F 0 "J16" H 5408 5681 50  0000 C CNN
+F 1 "DJ621-6.3" H 5408 5590 50  0000 C CNN
+F 2 "Connector:CONN_63824-1" H 5300 5500 50  0001 C CNN
+F 3 "~" H 5300 5500 50  0001 C CNN
+	1    5300 5500
+	1    0    0    -1
+$EndComp
+$Comp
+L Connector:Conn_01x01_Male J13
+U 1 1 62AE8D91
+P 5300 2450
+F 0 "J13" H 5408 2631 50  0000 C CNN
+F 1 "DJ621-6.3" H 5408 2540 50  0000 C CNN
+F 2 "Connector:CONN_63824-1" H 5300 2450 50  0001 C CNN
+F 3 "~" H 5300 2450 50  0001 C CNN
+	1    5300 2450
+	1    0    0    -1
+$EndComp
 $EndSCHEMATC

Commit message: tester up
Parts:
- removed J12, J13, J14, J15, J16: DJ621-6.3, Connector:CONN_63824-1, symbol Connector:Conn_01x01_Male
- added J25, J26, J27, J28, J29: DJ621-6.3, Connector:Knife_Terminal_6.3mm_P5.00mm_Vertical, symbol Connector:Conn_01x01_Male
Connections:
- net base_meas: now also J28.1 (Pin_1)
- net base_supp: now also J27.1 (Pin_1)
- net coll_meas: now also J26.1 (Pin_1)
- net coll_supp: now also J25.1 (Pin_1)
- net emitter: now also J29.1 (Pin_1)
Changed lines of the file:
@@
 Sheet 11 11
 Title ""
-Date ""
+Date "2022-04-25"
 Rev ""
 Comp ""
@@
 	6275 2450 5500 2450
 $Comp
-L Connector:Conn_01x01_Male J12
-U 1 1 62AE5BCB
+L Connector:Conn_01x01_Male J?
+U 1 1 627AAC5C
+P 5300 5500
+AR Path="/62558B2F/627AAC5C" Ref="J?"  Part="1"
+AR Path="/6253E238/627AAC5C" Ref="J29"  Part="1"
+F 0 "J29" H 5272 5432 50  0000 R CNN
+F 1 "DJ621-6.3" H 5272 5523 50  0000 R CNN
+F 2 "Connector:Knife_Terminal_6.3mm_P5.00mm_Vertical" H 5300 5500 50  0001 C CNN
+F 3 "~" H 5300 5500 50  0001 C CNN
+	1    5300 5500
+	1    0    0    -1
+$EndComp
+$Comp
+L Connector:Conn_01x01_Male J?
+U 1 1 627ACBD9
 P 5300 2150
-F 0 "J12" H 5408 2331 50  0000 C CNN
-F 1 "DJ621-6.3" H 5408 2240 50  0000 C CNN
-F 2 "Connector:CONN_63824-1" H 5300 2150 50  0001 C CNN
+AR Path="/62558B2F/627ACBD9" Ref="J?"  Part="1"
+AR Path="/6253E238/627ACBD9" Ref="J25"  Part="1"
+F 0 "J25" H 5272 2082 50  0000 R CNN
+F 1 "DJ621-6.3" H 5272 2173 50  0000 R CNN
+F 2 "Connector:Knife_Terminal_6.3mm_P5.00mm_Vertical" H 5300 2150 50  0001 C CNN
 F 3 "~" H 5300 2150 50  0001 C CNN
 	1    5300 2150
@@
 $EndComp
 $Comp
-L Connector:Conn_01x01_Male J14
-U 1 1 62AE5F58
+L Connector:Conn_01x01_Male J?
+U 1 1 627AD11A
+P 5300 2450
+AR Path="/62558B2F/627AD11A" Ref="J?"  Part="1"
+AR Path="/6253E238/627AD11A" Ref="J26"  Part="1"
+F 0 "J26" H 5272 2382 50  0000 R CNN
+F 1 "DJ621-6.3" H 5272 2473 50  0000 R CNN
+F 2 "Connector:Knife_Terminal_6.3mm_P5.00mm_Vertical" H 5300 2450 50  0001 C CNN
+F 3 "~" H 5300 2450 50  0001 C CNN
+	1    5300 2450
+	1    0    0    -1
+$EndComp
+$Comp
+L Connector:Conn_01x01_Male J?
+U 1 1 627AD706
 P 5300 3750
-F 0 "J14" H 5408 3931 50  0000 C CNN
-F 1 "DJ621-6.3" H 5408 3840 50  0000 C CNN
-F 2 "Connector:CONN_63824-1" H 5300 3750 50  0001 C CNN
+AR Path="/62558B2F/627AD706" Ref="J?"  Part="1"
+AR Path="/6253E238/627AD706" Ref="J27"  Part="1"
+F 0 "J27" H 5272 3682 50  0000 R CNN
+F 1 "DJ621-6.3" H 5272 3773 50  0000 R CNN
+F 2 "Connector:Knife_Terminal_6.3mm_P5.00mm_Vertical" H 5300 3750 50  0001 C CNN
 F 3 "~" H 5300 3750 50  0001 C CNN
 	1    5300 3750
@@
 $EndComp
 $Comp
-L Connector:Conn_01x01_Male J15
-U 1 1 62AE6B77
+L Connector:Conn_01x01_Male J?
+U 1 1 627ADCD8
 P 5300 4050
-F 0 "J15" H 5408 4231 50  0000 C CNN
-F 1 "DJ621-6.3" H 5408 4140 50  0000 C CNN
-F 2 "Connector:CONN_63824-1" H 5300 4050 50  0001 C CNN
+AR Path="/62558B2F/627ADCD8" Ref="J?"  Part="1"
+AR Path="/6253E238/627ADCD8" Ref="J28"  Part="1"
+F 0 "J28" H 5272 3982 50  0000 R CNN
+F 1 "DJ621-6.3" H 5272 4073 50  0000 R CNN
+F 2 "Connector:Knife_Terminal_6.3mm_P5.00mm_Vertical" H 5300 4050 50  0001 C CNN
 F 3 "~" H 5300 4050 50  0001 C CNN
 	1    5300 4050
 	1    0    0    -1
 $EndComp
-$Comp
-L Connector:Conn_01x01_Male J16
-U 1 1 62AE7081
-P 5300 5500
-F 0 "J16" H 5408 5681 50  0000 C CNN
-F 1 "DJ621-6.3" H 5408 5590 50  0000 C CNN
-F 2 "Connector:CONN_63824-1" H 5300 5500 50  0001 C CNN
-F 3 "~" H 5300 5500 50  0001 C CNN
-	1    5300 5500
-	1    0    0    -1
-$EndComp
-$Comp
-L Connector:Conn_01x01_Male J13
-U 1 1 62AE8D91
-P 5300 2450
-F 0 "J13" H 5408 2631 50  0000 C CNN
-F 1 "DJ621-6.3" H 5408 2540 50  0000 C CNN
-F 2 "Connector:CONN_63824-1" H 5300 2450 50  0001 C CNN
-F 3 "~" H 5300 2450 50  0001 C CNN
-	1    5300 2450
-	1    0    0    -1
-$EndComp
