File: Bipolar_transistor_tester_1.0/Bipolar_transistor_tester_1.0.sch (KiCad schematic (older format))
At the start: 0 parts

Commit message: tester up
Parts:
- added R? (x2): 1k 1%, Resistor_SMD:R_0805_2012Metric, symbol Device:R
- added U1: CPC1977, OptoDevice:i4-PAC, symbol Relay_SolidState:CPC1977
- added U2: PVN012, Package_DIP:DIP-6_W7.62mm, symbol Relay_SolidState:PVN012
Connections:
- net GND: now also U2.4
- net base_current_meter/in-: now also U1.2
- net measured transistor/base_supp: now also U1.1
- new net: R?.2, U2.1
- new net: R?.2, U1.4
- new net 4_com_an: R?.1, R?.1
- new net 4_rp1: U1.3
- new net 4_rp2: U2.2
- new net emitter_current_meter/in: U2.6
- no-connect marks 0 -> 1

Commit message: tester up
Parts:
- added H1, H2, H3, H4, H5, H6: MountingHole, MountingHole:MountingHole_3.2mm_M3, symbol Mechanical:MountingHole
- gave numbers to parts that had none: 2
Changed lines of the file:
@@
 Sheet 1 11
 Title ""
-Date ""
+Date "2022-04-25"
 Rev ""
 Comp ""
@@
 F1 "emitter_cur_meter.sch" 50
 F2 "in" I L 5500 5750 50
-F3 "gnd" I L 5500 6050 50
+F3 "to_gnd" I L 5500 6050 50
 $EndSheet
 $Sheet
@@
 P 4650 5100
 AR Path="/62559320/62871593" Ref="R?"  Part="1"
-AR Path="/62871593" Ref="R?"  Part="1"
-F 0 "R?" V 4443 5100 50  0000 C CNN
+AR Path="/62871593" Ref="R1"  Part="1"
+F 0 "R1" V 4443 5100 50  0000 C CNN
 F 1 "1k 1%" V 4534 5100 50  0000 C CNN
 F 2 "Resistor_SMD:R_0805_2012Metric" V 4580 5100 50  0001 C CNN
@@
 P 4650 5650
 AR Path="/62559320/628792CA" Ref="R?"  Part="1"
-AR Path="/628792CA" Ref="R?"  Part="1"
-F 0 "R?" V 4443 5650 50  0000 C CNN
+AR Path="/628792CA" Ref="R2"  Part="1"
+F 0 "R2" V 4443 5650 50  0000 C CNN
 F 1 "1k 1%" V 4534 5650 50  0000 C CNN
 F 2 "Resistor_SMD:R_0805_2012Metric" V 4580 5650 50  0001 C CNN
@@
 Text GLabel 4600 6000 0    50   Input ~ 0
 4_rp2
+$Comp
+L Mechanical:MountingHole H1
+U 1 1 626E66A2
+P -1200 2100
+F 0 "H1" H -1100 2146 50  0000 L CNN
+F 1 "MountingHole" H -1100 2055 50  0000 L CNN
+F 2 "MountingHole:MountingHole_3.2mm_M3" H -1200 2100 50  0001 C CNN
+F 3 "~" H -1200 2100 50  0001 C CNN
+	1    -1200 2100
+	1    0    0    -1
+$EndComp
+$Comp
+L Mechanical:MountingHole H2
+U 1 1 626E80C8
+P -1200 2400
+F 0 "H2" H -1100 2446 50  0000 L CNN
+F 1 "MountingHole" H -1100 2355 50  0000 L CNN
+F 2 "MountingHole:MountingHole_3.2mm_M3" H -1200 2400 50  0001 C CNN
+F 3 "~" H -1200 2400 50  0001 C CNN
+	1    -1200 2400
+	1    0    0    -1
+$EndComp
+$Comp
+L Mechanical:MountingHole H3
+U 1 1 626E8367
+P -1200 2700
+F 0 "H3" H -1100 2746 50  0000 L CNN
+F 1 "MountingHole" H -1100 2655 50  0000 L CNN
+F 2 "MountingHole:MountingHole_3.2mm_M3" H -1200 2700 50  0001 C CNN
+F 3 "~" H -1200 2700 50  0001 C CNN
+	1    -1200 2700
+	1    0    0    -1
+$EndComp
+$Comp
+L Mechanical:MountingHole H4
+U 1 1 626E870D
+P -1200 3000
+F 0 "H4" H -1100 3046 50  0000 L CNN
+F 1 "MountingHole" H -1100 2955 50  0000 L CNN
+F 2 "MountingHole:MountingHole_3.2mm_M3" H -1200 3000 50  0001 C CNN
+F 3 "~" H -1200 3000 50  0001 C CNN
+	1    -1200 3000
+	1    0    0    -1
+$EndComp
+$Comp
+L Mechanical:MountingHole H5
+U 1 1 6273A0A9
+P -1200 3300
+F 0 "H5" H -1100 3346 50  0000 L CNN
+F 1 "MountingHole" H -1100 3255 50  0000 L CNN
+F 2 "MountingHole:MountingHole_3.2mm_M3" H -1200 3300 50  0001 C CNN
+F 3 "~" H -1200 3300 50  0001 C CNN
+	1    -1200 3300
+	1    0    0    -1
+$EndComp
+$Comp
+L Mechanical:MountingHole H6
+U 1 1 6273A0AF
+P -1200 3600
+F 0 "H6" H -1100 3646 50  0000 L CNN
+F 1 "MountingHole" H -1100 3555 50  0000 L CNN
+F 2 "MountingHole:MountingHole_3.2mm_M3" H -1200 3600 50  0001 C CNN
+F 3 "~" H -1200 3600 50  0001 C CNN
+	1    -1200 3600
+	1    0    0    -1
+$EndComp
 $EndSCHEMATC

Commit message: edit resistors cpc1977
Parts:
- R1: value 1k 1% -> 270
Changed lines of the file:
@@
 AR Path="/62871593" Ref="R1"  Part="1"
 F 0 "R1" V 4443 5100 50  0000 C CNN
-F 1 "1k 1%" V 4534 5100 50  0000 C CNN
+F 1 "270" V 4534 5100 50  0000 C CNN
 F 2 "Resistor_SMD:R_0805_2012Metric" V 4580 5100 50  0001 C CNN
 F 3 "~" H 4650 5100 50  0001 C CNN
