File: Old_Convertor_15v_to_20v:500v/Old_Convertor_15v_to_20v:500v.kicad_pcb (KiCad board)
At the start: 2 copper layers, 90 x 80 mm, 54 parts, among them J1 Screw_Terminal_01x04, J2 Conn_01x04_Male, Q1 IRF640NSTR, T1 Transfomer_1P_1S_custom, U1 OP177, U2 UC3845_DIP8, U3 DCP011515D, U4 ISO124P, U5 CPC1977, U6 CPC1977, U7 PVN012, U8 CPC1977, U9 CPC1977

Commit message: old_convertor done
Parts:
- removed PS1: TMV1215D, Converter_DCDC:Converter_DCDC_XP_POWER-IHxxxxSH_THT
- added U5: DCP011515D, Converter_DCDC:Converter_DCDC_DCP01xxxxD, F.Cu at (169.2, 145.0)
- D2: value 1.5K100A -> 1.5KE75A
- L1: value 4uH -> L
- R10: value 36k 1% -> 30k 1%
- moved C13 10.8 mm to (174.0, 146.5), turned to 180 degrees
- moved C12 9.68 mm to (164.0, 146.2)
- moved C14 3.68 mm to (174.0, 144.2)
- renumbered C7 to C10, C12 to C11, C14 to C12, C9 to C13, C13 to C14, C6 to C5, C5 to C6, C8 to C7, C10 to C8, C11 to C9, R17 to R18, U9 to U10, U5 to U6, U6 to U7, U7 to U8, U8 to U9
Connections:
- C12 pad 1: Net-(C14-Pad1) -> +15V
- C12 pad 2: GND2 -> GND
- C13 pad 1: +15V -> Net-(C13-Pad1)
- C13 pad 2: GND -> GND2
- C14 pad 1: Net-(C13-Pad1) -> Net-(C14-Pad1)
Routing:
- net GND2: track 116.8 -> 132.1 mm
- net Net-(C13-Pad1): track 18.5 -> 23.3 mm
- net Net-(C14-Pad1): track 16.5 -> 20.7 mm
- net +15V: track 119.6 -> 117.1 mm
