File: Convertor_15v_to_20v:500v/Convertor_15v_to_20v:500v.sch (KiCad schematic (older format))
At the start: 54 parts, among them J1 Screw_Terminal_01x04, J2 Conn_01x04_Male, Q1 IRF640NSTR, T1 Transfomer_1P_1S_custom, U1 OP177, U10 CPC1977, U2 UC3845_DIP8, U3 DCP011515D, U4 ISO124P, U5 DCP011515D, U6 CPC1977, U7 CPC1977, U8 PVN012, U9 CPC1977

Commit message: tester up
Parts:
- removed U5: DCP011515D, Converter_DCDC:Converter_DCDC_DCP01xxxxD, symbol Converter_DCDC:DCP01xxxxD
- added PS1: TMV1215D, Converter_DCDC:Converter_DCDC_XP_POWER-IHxxxxSH_THT, symbol Converter_DCDC:IA0503S
- R10: value 30k 1% -> 36k 1%
- renumbered C8 to C10, C9 to C11, C11 to C12, C14 to C13, C12 to C14, C6 to C5, C5 to C6, C10 to C7, C7 to C8, C13 to C9, R18 to R17, U6 to U5, U7 to U6, U8 to U7, U9 to U8, U10 to U9
Connections:
- net +15V: now also C9.1, PS1.1 (+Vin); no longer C14.1
- net GND: now also C9.2, PS1.2 (-Vin); no longer C14.2
- net GND2: now also C14.2, PS1.5 (0V); no longer C9.2
- net at U4.1 (+Vs1): now also C13.1, PS1.6 (+Vout); no longer C9.1
- net at U4.2 (-Vs1): now also C14.1, PS1.4 (-Vout); no longer C13.1
- no-connect marks 5 -> 3
Other:
- moved on the sheet: C13, C14, C9

Commit message: tester up
Parts:
- R7: value 0.2 -> 0.2 0.25W
- U2: value UC3845_DIP8 -> UC3845
Changed lines of the file:
@@
 P 3400 2900
 F 0 "U2" H 3400 3481 50  0000 C CNN
-F 1 "UC3845_DIP8" H 3400 3390 50  0000 C CNN
+F 1 "UC3845" H 3400 3390 50  0000 C CNN
 F 2 "Package_DIP:DIP-8_W7.62mm" H 3400 2400 50  0001 C CNN
 F 3 "http://www.ti.com/lit/ds/symlink/uc3842.pdf" H 3400 2900 50  0001 C CNN
@@
 P 4700 3325
 F 0 "R7" H 4630 3279 50  0000 R CNN
-F 1 "0.2" H 4630 3370 50  0000 R CNN
+F 1 "0.2 0.25W" H 4630 3370 50  0000 R CNN
 F 2 "Resistor_THT:R_Axial_DIN0207_L6.3mm_D2.5mm_P10.16mm_Horizontal" V 4630 3325 50  0001 C CNN
 F 3 "~" H 4700 3325 50  0001 C CNN

Commit message: Convertor edit dcp011515 to tmv1215d
Parts:
- removed U3: DCP011515D, Converter_DCDC:Converter_DCDC_DCP01xxxxD, symbol Converter_DCDC:DCP01xxxxD
- added PS2: TMV1215D, Converter_DCDC:Converter_DCDC_XP_POWER-IHxxxxSH_THT, symbol Converter_DCDC:IA0503S
Connections:
- net GND: now also PS2.2 (-Vin), PS2.5 (0V)
- net at C8.1, U1.7 (V+), U4.5 (+Vs2): now also PS2.6 (+Vout)
- net at C7.1, U1.4 (V-), U4.6 (-Vs2): now also PS2.4 (-Vout)
- net +15V renamed +12V
- net +12V: now also PS2.1 (+Vin)
- no-connect marks 3 -> 1
Other:
- note added: "Трасформатор Т1\nВыводы 1-5: 18 витков, 0.6мм; 6-10: 90 витков, 0.3мм.\nСердечнин Epcos N87 E25/13/7, нужно создать зазор в сердечнике 0.3мм \n"
- note removed: "Трасформатор Т1\nВыводы 1-5: 18 витков, 0.6мм; 6-10: 90 витков, 0.2мм.\nСердечнин Epcos N87 E25/13/7, нужно создать зазор в сердечнике 0.3мм \n"
- moved on the sheet: C13, C14, C5, C7, C8, C9, PS1

Commit message: up
Parts:
- Q1: value IRF640NSTR -> IRFR320
Changed lines of the file:
@@
 P 4600 2700
 F 0 "Q1" H 4804 2746 50  0000 L CNN
-F 1 "IRF640NSTR" H 4804 2655 50  0000 L CNN
+F 1 "IRFR320" H 4804 2655 50  0000 L CNN
 F 2 "Package_TO_SOT_SMD:TO-252-2" H 4850 2625 50  0001 L CIN
 F 3 "http://www.irf.com/product-info/datasheets/data/irf540n.pdf" H 4600 2700 50  0001 L CNN
