File: Logic_signal_amplifier/Logic_signal_amplifier.kicad_pcb (KiCad board)
At the start: 2 copper layers, 55 x 120 mm, 24 parts, among them J1 Conn_01x07_Male, J10 KF2510_5pin, J11 KF2510_5pin, J12 KF2510_6pin, J13 KF2510_4pin, J14 Screw_Terminal_01x02, J2 Conn_01x07_Male, J3 Conn_01x07_Male, J4 Conn_01x07_Male, J5 Conn_01x06_Male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

Commit message: up
Parts:
- added J15: KF2510_4pin, Connector_KF2510:KF2510_4pin, F.Cu at (143.7, 132.2)
- added J16: KF2510_4pin, Connector_KF2510:KF2510_4pin, F.Cu at (133.3, 146.0)
- added U6: ULN2004A, Package_SO:SOIC-16_4.55x10.3mm_P1.27mm, F.Cu at (112.0, 152.1)
- J12: value KF2510_6pin -> KF2510_5pin; footprint Connector_KF2510:KF2510_6pin -> Connector_KF2510:KF2510_5pin
- J13: value KF2510_4pin -> KF2510_5pin; footprint Connector_KF2510:KF2510_4pin -> Connector_KF2510:KF2510_5pin
- J14: value Screw_Terminal_01x02 -> KF2510_6pin; footprint TerminalBlock_Phoenix:TerminalBlock_Phoenix_MKDS-1,5-2-5.08_1x02_P5.08mm_Horizontal -> Connector_KF2510:KF2510_6pin
- J6: value KF2510_6pin -> KF2510_3pin; footprint Connector_KF2510:KF2510_6pin -> Connector_KF2510:KF2510_3pin
- J7: value KF2510_6pin -> Screw_Terminal_01x02; footprint Connector_KF2510:KF2510_6pin -> TerminalBlock_Phoenix:TerminalBlock_Phoenix_MKDS-1,5-2-5.08_1x02_P5.08mm_Horizontal
- J8, J9: value KF2510_5pin -> KF2510_6pin; footprint Connector_KF2510:KF2510_5pin -> Connector_KF2510:KF2510_6pin
- moved J6 107.5 mm to (99.2, 146.0)
- moved J14 77.0 mm to (133.3, 116.4), turned to 0 degrees
- moved J7 30.0 mm to (119.5, 38.5), turned to 180 degrees
- moved J13 28.0 mm to (143.3, 104.2)
- moved J8 26.5 mm to (132.7, 43.9)
- moved J9 24.5 mm to (143.6, 56.3)
- moved J12 23.5 mm to (132.8, 92.9)
- moved J11 23.4 mm to (143.6, 80.8)
- moved J10 22.5 mm to (132.7, 70.4)
- moved H3 11.0 mm to (97.0, 158.0)
- moved H4 11.0 mm to (144.0, 158.0)
- moved H1 1.00 mm to (97.0, 36.0)
- moved H2 1.00 mm to (144.0, 36.0)
Connections:
- J10 pad 2: 5_bcm1 -> 3_ccm1
- J10 pad 3: 5_bcm2 -> 3_ccm2
- J10 pad 4: 5_bcm3 -> 3_ccm3
- J10 pad 5: 5_bcm4 -> 3_ccm4
- J11 pad 2: 6_bvs1 -> 4_ecm1
- J11 pad 3: 6_bvs2 -> 4_ecm2
- J11 pad 4: 6_bvs3 -> 4_rp1
- J11 pad 5: 6_bvs4 -> 4_rp2
- J12 pad 2: 7_br1 -> 5_bcm1
- J12 pad 3: 7_br2 -> 5_bcm2
- J12 pad 4: 7_br3 -> 5_bcm3
- J12 pad 5: 7_br4 -> 5_bcm4
- J13 pad 2: 8_cbvm1 -> 6_bvs1
- J13 pad 3: 8_cbvm2 -> 6_bvs2
- J13 pad 4: 8_cbvm3 -> 6_bvs3
- J14 pad 2: GND -> 7_br1
- J6 pad 1: +5V -> Net-(J6-Pad1)
- J6 pad 2: 1_ccs1 -> Net-(J6-Pad2)
- J6 pad 3: 1_ccs2 -> Net-(J6-Pad3)
- J7 pad 2: 2_bcs1 -> GND
- J8 pad 2: 3_ccm1 -> 1_ccs1
- J8 pad 3: 3_ccm2 -> 1_ccs2
- J8 pad 4: 3_ccm3 -> 1_ccs3
- J8 pad 5: 3_ccm4 -> 1_ccs4
- J9 pad 2: 4_ecm1 -> 2_bcs1
- J9 pad 3: 4_ecm2 -> 2_bcs2
- J9 pad 4: 4_rp1 -> 2_bcs3
- J9 pad 5: 4_rp2 -> 2_bcs4
Routing:
- net +5V: track 295.4 -> 336.1 mm, vias 5 -> 6
- net GND: track 112.6 -> 135.1 mm, vias 5 -> 6
- net set_negativ: track 0.00 -> 19.5 mm
- net set_positive: track 0.00 -> 18.9 mm
- net dac_relay: track 0.00 -> 18.4 mm
- net Net-(J6-Pad1): track 0.00 -> 10.2 mm
- net Net-(J6-Pad3): track 0.00 -> 9.92 mm
- net Net-(J6-Pad2): track 0.00 -> 9.71 mm
Other:
- board size 55 x 120 mm -> 55 x 130 mm
- board text added: "40-500V"
- board text added: "Rev: 1.1"
- board text removed: "Rev: 1.0"
