File: Logic_signal_amplifier/Logic_signal_amplifier.sch (KiCad schematic (older format))
At the start: 24 parts, among them J1 Conn_01x07_Male, J10 KF2510_5pin, J11 KF2510_5pin, J12 KF2510_6pin, J13 KF2510_4pin, J14 Screw_Terminal_01x02, J2 Conn_01x07_Male, J3 Conn_01x07_Male, J4 Conn_01x07_Male, J5 Conn_01x06_Male, J6 KF2510_6pin, J7 KF2510_6pin, J8 KF2510_5pin, J9 KF2510_5pin, U1 ULN2004A, U2 ULN2004A, U3 ULN2004A, U4 ULN2004A, U5 ULN2004A

Commit message: up
Parts:
- added J16: KF2510_4pin, Connector_KF2510:KF2510_4pin, symbol Connector:Conn_01x04_Male
- added J6: KF2510_3pin, Connector_KF2510:KF2510_3pin, symbol Connector:Conn_01x03_Male
- added U6: ULN2004A, Package_SO:SOIC-16_4.55x10.3mm_P1.27mm, symbol Transistor_Array:ULN2004A
- renumbered J8 to J10, J9 to J11, J10 to J12, J11 to J13, J12 to J14, J13 to J15, J14 to J7, J6 to J8, J7 to J9
Connections:
- net +5V: now also J16.1 (Pin_1), U6.9 (COM)
- net GND: now also U6.8 (GND)
- new net: J6.1 (Pin_1), U6.1 (I1)
- new net: J6.2 (Pin_2), U6.2 (I2)
- new net: J6.3 (Pin_3), U6.3 (I3)
- new net dac_relay: J16.2 (Pin_2), U6.16 (O1)
- new net set_negativ: J16.4 (Pin_4), U6.14 (O3)
- new net set_positive: J16.3 (Pin_3), U6.15 (O2)
- no-connect marks 2 -> 10
Other:
- moved on the sheet: C1, H1, H2, H3, H4, J1, J10, J11, J12, J13, J14, J15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
